File: Borg/01/01.kicad_pcb (KiCad board)
At the start: 2 copper layers, 0 parts

Commit message: Some updates
Parts:
- added svg2mod: G***, borg:Borg.Edge.01, F.Cu at (141.0, 101.0)
- added svg2mod: G***, borg:Borg.Cu.01, F.Cu at (214.0, 91.4)
Other:
- board outline added: 98.7 x 98.6 mm
Changed lines of the file:
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@@
-(kicad_pcb (version 4) (host pcbnew 4.0.1-3.201512221402+6198~38~ubuntu14.04.1-stable)
+(kicad_pcb (version 20171130) (host pcbnew 6.0.0-rc1-unknown-5b3202d~66~ubuntu16.04.1)
   (general
-    (links 0)
-    (no_connects 0)
-    (area 104.572999 74.854999 178.510001 123.265001)
     (thickness 1.6)
     (drawings 17)
     (tracks 0)
     (zones 0)
-    (modules 0)
+    (modules 2)
     (nets 1)
   )
@@
     (zone_45_only no)
     (trace_min 0.1524)
-    (segment_width 0.1524)
-    (edge_width 0.1524)
     (via_size 0.6858)
     (via_drill 0.3302)
@@
     (uvia_min_size 0)
     (uvia_min_drill 0)
+    (edge_width 0.1524)
+    (segment_width 0.1524)
     (pcb_text_width 0.1524)
     (pcb_text_size 1.016 1.016)
@@
       (layerselection 0x310fc_80000001)
       (usegerberextensions true)
+      (usegerberattributes false)
+      (usegerberadvancedattributes false)
+      (creategerberjobfile false)
       (excludeedgelayer true)
       (linewidth 0.100000)
@@
       (hpglpennumber 1)
       (hpglpenspeed 20)
-      (hpglpendiameter 15)
-      (hpglpenoverlay 2)
+      (hpglpendiameter 15.000000)
       (psnegative false)
       (psa4output false)
@@
       (drillshape 0)
       (scaleselection 1)
-      (outputdirectory gerbers))
+      (outputdirectory "gerbers"))
   )
   (net 0 "")
@@
     (uvia_drill 0.3302)
   )
+  (module borg:Borg.Edge.01 (layer F.Cu)
+    (at 140.97 100.965)
+    (descr "Imported from Borg_Base.svg")
+    (tags svg2mod)
+    (attr smd)
+    (fp_text reference svg2mod (at 0 -52.32336) (layer F.SilkS) hide
+      (effects (font (size 1.524 1.524) (thickness 0.3048)))
+    )
+    (fp_text value G*** (at 0 52.32336) (layer F.SilkS) hide
+      (effects (font (size 1.524 1.524) (thickness 0.3048)))
+    )
+    (fp_line (start -49.347716 49.27536) (end -49.347716 -49.27536) (layer Edge.Cuts) (width 0.285533))
+    (fp_line (start 49.347716 49.27536) (end -49.347716 49.27536) (layer Edge.Cuts) (width 0.285533))
+    (fp_line (start 49.347716 -49.27536) (end 49.347716 49.27536) (layer Edge.Cuts) (width 0.285533))
+    (fp_line (start -49.347716 -49.27536) (end 49.347716 -49.27536) (layer Edge.Cuts) (width 0.285533))
+  )
+  (module borg:Borg.Cu.01 (layer F.Cu)
+    (at 213.995 91.44)
+    (descr "Imported from Borg_Base.svg")
+    (tags svg2mod)
+    (attr smd)
+    (fp_text reference svg2mod (at 0 -3.048) (layer F.SilkS) hide
+      (effects (font (size 1.524 1.524) (thickness 0.3048)))
+    )
+    (fp_text value G*** (at 0 3.048) (layer F.SilkS) hide
+      (effects (font (size 1.524 1.524) (thickness 0.3048)))
+    )
+  )
   (gr_circle (center 117.348 76.962) (end 118.618 76.962) (layer Dwgs.User) (width 0.15))
