File: Orange/02/01.kicad_pcb (KiCad board)
At the start: 2 copper layers, 0 parts

Commit message: some updates
Parts:
- added svg2mod: G***, orange:orange2.All.02, F.Cu at (134.6, 99.1)
Other:
- board outline added: 52.4 x 40.6 mm
