File: wemos-microbit/wemos-01.kicad_pcb (KiCad board)
At the start: 2 copper layers, 54.6 x 36.8 mm, 3 parts, among them P1 CONN_01X08, P2 CONN_01X08

Commit message: Some updates
Parts:
- removed REF**: Microbit_PCB_Connector, wemos_microbit:Microbit_PCB_Connector
- added J1: Microbit_01X25, wemos_microbit:Microbit_PCB_Connector, F.Cu at (139.7, 116.8)
Connections:
- P2 pad 2: /D8 -> (no net)
- P2 pad 3: /D7 -> (no net)
- P2 pad 4: /D6 -> (no net)
- P2 pad 5: /D5 -> (no net)
Routing:
- net /D0: track 0.00 -> 23.1 mm
Other:
- board size 54.6 x 36.8 mm -> 52 x 35.9 mm
