File: MazBasica/001/Arduino_As_Uno.sch (KiCad schematic (older format))
At the start: 23 parts, among them P1 Power, P2 Analog, P3 Digital, P4 Digital, P5 CONN_01X01, P6 CONN_01X01, P7 CONN_01X01, P8 CONN_01X01, SW1 SW_Push, SW2 SW_Push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

Commit message: some changes mazbasica
Parts:
- removed P5, P6, P7, P8: CONN_01X01, Socket_Arduino_Uno:Arduino_1pin, symbol conn:CONN_01X01
- removed SW3: SW_Push, symbol switches:SW_Push
- removed U1: DHT11, symbol sensors:DHT11
- added J1: CONN_01X04, Connector_PinHeader_2.54mm:PinHeader_1x04_P2.54mm_Vertical, symbol conn:CONN_01X04
- added J2, J3: CONN_01X03, Connector_PinHeader_2.54mm:PinHeader_1x03_P2.54mm_Vertical, symbol conn:CONN_01X03
- added J4: CONN_01X06, Connector_PinHeader_2.54mm:PinHeader_1x06_P2.54mm_Vertical, symbol conn:CONN_01X06
- added J5: CONN_01X01, Connector_PinHeader_2.54mm:PinHeader_1x01_P2.54mm_Vertical, symbol conn:CONN_01X01
- added R7: 1k, Resistor_SMD:R_1206_3216Metric_Pad1.39x1.80mm_HandSolder, symbol device:R_Small
- BZ1: footprint (none) -> Buzzer_Beeper:Buzzer_12x9.5RM7.6
- LED1, LED2, LED3: footprint (none) -> Socket_Arduino_Uno:PL9823
- R1: footprint (none) -> OptoDevice:R_LDR_4.9x4.2mm_P2.54mm_Vertical
- R2, R3, R4, R5: footprint (none) -> Resistor_SMD:R_1206_3216Metric_Pad1.39x1.80mm_HandSolder
- R6: value 330 -> 2k; footprint (none) -> Resistor_SMD:R_1206_3216Metric_Pad1.39x1.80mm_HandSolder
- RV1: footprint (none) -> Potentiometer_THT:Potentiometer_Bourns_PTV09A-1_Single_Vertical
- SW1, SW2: footprint (none) -> Button_Switch_THT:SW_PUSH_6mm
Connections:
- net +5V: now also LED1.2 (VCC), LED2.2 (VCC), LED3.2 (VCC), J1.1 (P1), J2.2 (P2), J3.2 (P2), J4.2 (P2); no longer R6.1
- net 0(Rx): now also J4.4 (P4)
- net 1(Tx): now also R6.1, R7.1
- net 2: now also J1.2 (P2)
- net 3(**): now also BZ1.1 (-)
- net 4: no longer R4.2, SW1.2
- net 5(**): now also J2.1 (P1)
- net 6(**): now also J3.1 (P1)
- net 7: no longer R5.2, SW2.2
- net A2: now also R4.2, SW1.2
- net A3: now also R5.2, SW2.2
- net GND: now also LED1.3 (GND), LED2.3 (GND), LED3.3 (GND), R6.2, J1.4 (P4), J2.3 (P3), J3.3 (P3), J4.3 (P3)
- net Reset: now also J5.1 (P1)
- new net: J4.5 (P5), R7.2
- no-connect marks 6 -> 5
Other:
- note added: "* BLUETOOTH 0"
- note added: "* BLUETOOTH 1"
- note added: "* BUZZER"
- note added: "* NEOPIXEL"
- note added: "* SERVO A"
- note added: "* SERVO B"
- note added: "BLUETOOTH"
- note added: "BUTTON A"
- note added: "BUTTON A *"
- note added: "BUTTON B"
- note added: "BUTTON B *"
- note added: "BUZZER"
- note added: "DHT11"
- note added: "LDR"
- note added: "LDR *"
- note added: "NEOPIXEL"
- note added: "POT"
- note added: "POT *"
- note added: "SERVO A"
- note added: "SERVO B"
- note removed: "Holes"
- moved on the sheet: BZ1, LED1, LED2, LED3, R1, R2, R3, R4, R5, RV1, SW1, SW2

Commit message: Updates
Parts:
- BZ1: symbol device:Buzzer -> Arduino_As_Uno-rescue:Buzzer-device
- J1: symbol conn:CONN_01X04 -> Arduino_As_Uno-rescue:CONN_01X04-conn
- J2, J3: symbol conn:CONN_01X03 -> Arduino_As_Uno-rescue:CONN_01X03-conn
- J4, P2: symbol conn:CONN_01X06 -> Arduino_As_Uno-rescue:CONN_01X06-conn
- J5: symbol conn:CONN_01X01 -> Arduino_As_Uno-rescue:CONN_01X01-conn
- LED1, LED2, LED3: symbol pl9823:PL9823 -> Arduino_As_Uno-rescue:PL9823-pl9823
- P1, P4: symbol conn:CONN_01X08 -> Arduino_As_Uno-rescue:CONN_01X08-conn
- P3: symbol conn:CONN_01X10 -> Arduino_As_Uno-rescue:CONN_01X10-conn
- R1: symbol device:RES_PHOTO_LDR -> Arduino_As_Uno-rescue:RES_PHOTO_LDR-device
- R2, R3, R4, R5, R6, R7: symbol device:R_Small -> Arduino_As_Uno-rescue:R_Small-device
- RV1: symbol device:POT -> Arduino_As_Uno-rescue:POT-device
- SW1, SW2: symbol switches:SW_Push -> Arduino_As_Uno-rescue:SW_Push-switches
Changed lines of the file:
@@
 Shield for Arduino that uses\nthe same pin disposition\nlike "Uno" board Rev 3.
 $Comp
-L conn:CONN_01X08 P1
+L Arduino_As_Uno-rescue:CONN_01X08-conn P1
 U 1 1 56D70129
 P 9600 1950
@@
 $EndComp
 $Comp
-L conn:CONN_01X06 P2
+L Arduino_As_Uno-rescue:CONN_01X06-conn P2
 U 1 1 56D70DD8
 P 9600 2750
@@
 $EndComp
 $Comp
-L conn:CONN_01X08 P4
+L Arduino_As_Uno-rescue:CONN_01X08-conn P4
 U 1 1 56D7164F
 P 10000 2650
@@
 	9400 3000 8900 3000
 $Comp
-L conn:CONN_01X10 P3
+L Arduino_As_Uno-rescue:CONN_01X10-conn P3
 U 1 1 56D721E0
 P 10000 1650
@@
 1
 $Comp
-L switches:SW_Push SW1
+L Arduino_As_Uno-rescue:SW_Push-switches SW1
 U 1 1 5C3FE3F4
 P 4900 950
@@
 $EndComp
 $Comp
-L switches:SW_Push SW2
+L Arduino_As_Uno-rescue:SW_Push-switches SW2
 U 1 1 5C3FEF50
 P 4900 1450
@@
 $EndComp
 $Comp
-L pl9823:PL9823 LED2
+L Arduino_As_Uno-rescue:PL9823-pl9823 LED2
 U 1 1 5C4049A9
 P 2000 2275
@@
 $EndComp
 $Comp
-L device:RES_PHOTO_LDR R1
+L Arduino_As_Uno-rescue:RES_PHOTO_LDR-device R1
 U 1 1 5C40A3DE
 P 2025 4550
@@
 	2650 2075 2500 2075
 $Comp
-L pl9823:PL9823 LED3
+L Arduino_As_Uno-rescue:PL9823-pl9823 LED3
 U 1 1 5C40D6B4
 P 2000 3275
@@
 A0
 $Comp
-L device:R_Small R2
+L Arduino_As_Uno-rescue:R_Small-device R2
 U 1 1 5C41A6BC
 P 2250 4150
@@
 $EndComp
 $Comp
-L device:R_Small R3
+L Arduino_As_Uno-rescue:R_Small-device R3
 U 1 1 5C435952
 P 2650 6725
@@
 	2175 5750 2300 5750
 $Comp
-L device:POT RV1
+L Arduino_As_Uno-rescue:POT-device RV1
 U 1 1 5C4091EE
 P 2025 5750
@@
 Connection ~ 5225 950
 $Comp
-L device:R_Small R4
+L Arduino_As_Uno-rescue:R_Small-device R4
 U 1 1 5C4826B8
 P 5450 950
@@
 $EndComp
 $Comp
-L device:R_Small R5
+L Arduino_As_Uno-rescue:R_Small-device R5
 U 1 1 5C4830EC
 P 5450 1450
@@
 $EndComp
 $Comp
-L device:Buzzer BZ1
+L Arduino_As_Uno-rescue:Buzzer-device BZ1
 U 1 1 5C409638
 P 4800 2050
@@
 $EndComp
 $Comp
-L pl9823:PL9823 LED1
+L Arduino_As_Uno-rescue:PL9823-pl9823 LED1
 U 1 1 5C403566
 P 2000 1275
@@
 $EndComp
 $Comp
-L conn:CONN_01X04 J1
+L Arduino_As_Uno-rescue:CONN_01X04-conn J1
 U 1 1 5C438DD4
 P 2200 7000
@@
 BUTTON B *
 $Comp
-L conn:CONN_01X03 J2
+L Arduino_As_Uno-rescue:CONN_01X03-conn J2
 U 1 1 5C4C4E51
 P 5200 3350
@@
 $EndComp
 $Comp
-L conn:CONN_01X03 J3
+L Arduino_As_Uno-rescue:CONN_01X03-conn J3
 U 1 1 5C4C562B
 P 5200 3875
@@
 * SERVO B
 $Comp
-L conn:CONN_01X06 J4
+L Arduino_As_Uno-rescue:CONN_01X06-conn J4
 U 1 1 5C4E57FD
 P 5800 5025
@@
 $EndComp
 $Comp
-L conn:CONN_01X01 J5
+L Arduino_As_Uno-rescue:CONN_01X01-conn J5
 U 1 1 5C4E6C74
 P 5800 5500
@@
 	5600 5175 5225 5175
 $Comp
-L device:R_Small R7
+L Arduino_As_Uno-rescue:R_Small-device R7
 U 1 1 5C4F77B7
 P 5125 5175
@@
 Connection ~ 4900 5175
 $Comp
-L device:R_Small R6
+L Arduino_As_Uno-rescue:R_Small-device R6
 U 1 1 5C5045D7
 P 4900 5400
