File: MazBasica/001/Arduino_As_Uno.kicad_pcb (KiCad board)
At the start: 2 copper layers, 48.3 x 53.3 mm, 23 parts, among them J1 CONN_01X04, J2 CONN_01X03, J3 CONN_01X03, J4 CONN_01X06, J5 CONN_01X01, P1 Power, P2 Analog, P3 Digital, P4 Digital, SW1 SW_Push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

Commit message: Update
Parts:
- added svg2mod: G***, Mazbasica:Puro.01, F.Cu at (137.9, 87.6)
- added svg2mod: G***, Mazbasica:IntLetters.01, F.Cu at (139.3, 87.1)
- added svg2mod: G***, Mazbasica:logoSin.03, F.Cu at (137.7, 87.6)
- added svg2mod: G***, Mazbasica:logoSinOut.01, F.Cu at (137.7, 87.6)
- added svg2mod: G***, Mazbasica:logoSinIn.01, F.Cu at (137.7, 87.6)
- added svg2mod: G***, Mazbasica:SinaloaCuMask.01, F.Cu at (137.7, 87.5)
- moved LED3 18.5 mm to (147.8, 99.7)
- moved LED1 17.3 mm to (130.0, 99.7)
- moved J3 2.54 mm to (121.2, 97.2)
- moved R3 2.29 mm to (152.3, 92.1)
- moved R6 2.29 mm to (152.3, 85.7)
- moved R7 2.29 mm to (152.3, 88.9)
- moved R5 2.25 mm to (129.4, 109.9)
- moved LED2 2.01 mm to (138.9, 99.7)
- moved J2 1.91 mm to (121.2, 102.9)
- moved R2 1.91 mm to (140.8, 112.4)
- moved BZ1 1.27 mm to (118.0, 85.7)
- moved SW1 1.27 mm to (114.8, 113.0)
- moved SW2 1.27 mm to (126.2, 113.0)
- moved J5 0.53 mm to (158.6, 82.7)
- moved R4 0.51 mm to (118.5, 109.9)
- renumbered R1 to LDR
Other:
- board text added: "A"
- board text added: "B"
- board text added: "BLUETOOTH"
- board text added: "DHT11"
- board text added: "EDU BASICA"
- board text added: "S1"
- board text added: "S2"
- board text added: "v1.0"

Commit message: changes
Parts:
- added svg2mod: G***, Mazbasica:demo_win, F.Cu at (130.7, 80.0)
