File: ws2812b_reverse/Base/Base.sch (KiCad schematic (older format))
At the start: 0 parts

Commit message: Update
Parts:
- added U1: NeoReverse, neo-reverse:Neo-reverse_SMD_4Pin, symbol Neo_Reverse:NeoReverse
Connections:
- new net DIN: U1.4 (DIN)
- new net DOUT: U1.2 (DOUT)
- new net VDD: U1.1 (VDD)
- new net VSS: U1.3 (VSS)
Changed lines of the file:
@@
-EESchema Schematic File Version 2
-LIBS:power
-EELAYER 25 0
+EESchema Schematic File Version 4
+EELAYER 29 0
 EELAYER END
 $Descr USLetter 11000 8500
@@
 Comment4 ""
 $EndDescr
+Text GLabel 5075 2975 0    50   Input ~ 0
+VDD
+Text GLabel 5675 2975 2    50   Input ~ 0
+VSS
+$Comp
+L power:PWR_FLAG #FLG01
+U 1 1 5C49958D
+P 7825 2575
+F 0 "#FLG01" H 7825 2650 50  0001 C CNN
+F 1 "PWR_FLAG" H 7825 2748 50  0000 C CNN
+F 2 "" H 7825 2575 50  0001 C CNN
+F 3 "~" H 7825 2575 50  0001 C CNN
+	1    7825 2575
+	1    0    0    -1
+$EndComp
+Wire Wire Line
+	7825 2575 7825 2700
+$Comp
+L power:PWR_FLAG #FLG02
+U 1 1 5C499E58
+P 8225 2700
+F 0 "#FLG02" H 8225 2775 50  0001 C CNN
+F 1 "PWR_FLAG" H 8225 2873 50  0000 C CNN
+F 2 "" H 8225 2700 50  0001 C CNN
+F 3 "~" H 8225 2700 50  0001 C CNN
+	1    8225 2700
+	-1   0    0    1
+$EndComp
+Wire Wire Line
+	8225 2700 8225 2575
+Text GLabel 5675 3075 2    50   Input ~ 0
+DIN
+Text GLabel 7825 2700 3    50   Input ~ 0
+VSS
+Text GLabel 8225 2575 1    50   Input ~ 0
+VDD
+$Comp
+L Neo_Reverse:NeoReverse U1
+U 1 1 5C49DB8A
+P 5375 3025
+F 0 "U1" H 5375 3300 50  0000 C CNN
+F 1 "NeoReverse" H 5375 3209 50  0000 C CNN
+F 2 "neo-reverse:Neo-reverse_SMD_4Pin" H 5375 3025 50  0001 C CNN
+F 3 "" H 5375 3025 50  0001 C CNN
+	1    5375 3025
+	1    0    0    -1
+$EndComp
+Text GLabel 5075 3075 0    50   Input ~ 0
+DOUT
 $EndSCHEMATC

Commit message: Update
Parts:
- removed U1: NeoReverse, neo-reverse:Neo-reverse_SMD_4Pin, symbol Neo_Reverse:NeoReverse
- added U1: NeoReverse-Neo_Reverse, neo-reverse:Neo-reverse_SMD_4Pin, symbol Base-rescue:NeoReverse-Neo_Reverse
Connections:
- net VDD: now also U1.1 (VDD)
- net VSS: now also U1.3 (VSS)
Changed lines of the file:
@@
 EESchema Schematic File Version 4
+LIBS:Base-cache
 EELAYER 29 0
 EELAYER END
@@
 Comment4 ""
 $EndDescr
-Text GLabel 5075 2975 0    50   Input ~ 0
+Text GLabel 5125 1500 0    50   Input ~ 0
 VDD
-Text GLabel 5675 2975 2    50   Input ~ 0
+Text GLabel 5725 1600 2    50   Input ~ 0
 VSS
 $Comp
 L power:PWR_FLAG #FLG01
 U 1 1 5C49958D
-P 7825 2575
-F 0 "#FLG01" H 7825 2650 50  0001 C CNN
-F 1 "PWR_FLAG" H 7825 2748 50  0000 C CNN
-F 2 "" H 7825 2575 50  0001 C CNN
-F 3 "~" H 7825 2575 50  0001 C CNN
-	1    7825 2575
+P 9825 950
+F 0 "#FLG01" H 9825 1025 50  0001 C CNN
+F 1 "PWR_FLAG" H 9825 1123 50  0000 C CNN
+F 2 "" H 9825 950 50  0001 C CNN
+F 3 "~" H 9825 950 50  0001 C CNN
+	1    9825 950
 	1    0    0    -1
 $EndComp
 Wire Wire Line
-	7825 2575 7825 2700
+	9825 950  9825 1075
 $Comp
 L power:PWR_FLAG #FLG02
 U 1 1 5C499E58
-P 8225 2700
-F 0 "#FLG02" H 8225 2775 50  0001 C CNN
-F 1 "PWR_FLAG" H 8225 2873 50  0000 C CNN
-F 2 "" H 8225 2700 50  0001 C CNN
-F 3 "~" H 8225 2700 50  0001 C CNN
-	1    8225 2700
+P 10225 1075
+F 0 "#FLG02" H 10225 1150 50  0001 C CNN
+F 1 "PWR_FLAG" H 10225 1248 50  0000 C CNN
+F 2 "" H 10225 1075 50  0001 C CNN
+F 3 "~" H 10225 1075 50  0001 C CNN
+	1    10225 1075
 	-1   0    0    1
 $EndComp
 Wire Wire Line
-	8225 2700 8225 2575
-Text GLabel 5675 3075 2    50   Input ~ 0
-DIN
-Text GLabel 7825 2700 3    50   Input ~ 0
+	10225 1075 10225 950
+Text GLabel 9825 1075 3    50   Input ~ 0
 VSS
-Text GLabel 8225 2575 1    50   Input ~ 0
+Text GLabel 10225 950  1    50   Input ~ 0
 VDD
 $Comp
-L Neo_Reverse:NeoReverse U1
-U 1 1 5C49DB8A
-P 5375 3025
-F 0 "U1" H 5375 3300 50  0000 C CNN
-F 1 "NeoReverse" H 5375 3209 50  0000 C CNN
-F 2 "neo-reverse:Neo-reverse_SMD_4Pin" H 5375 3025 50  0001 C CNN
-F 3 "" H 5375 3025 50  0001 C CNN
-	1    5375 3025
+L Base-rescue:NeoReverse-Neo_Reverse U1
+U 1 1 5C4A5F1C
+P 5425 1550
+F 0 "U1" H 5425 1825 50  0000 C CNN
+F 1 "NeoReverse-Neo_Reverse" H 5425 1734 50  0000 C CNN
+F 2 "neo-reverse:Neo-reverse_SMD_4Pin" H 5425 1550 50  0001 C CNN
+F 3 "" H 5425 1550 50  0001 C CNN
+	1    5425 1550
 	1    0    0    -1
 $EndComp
-Text GLabel 5075 3075 0    50   Input ~ 0
-DOUT
 $EndSCHEMATC
