File: ws2812b_reverse/Base/Base.kicad_pcb (KiCad board)
At the start: 2 copper layers, 31.8 x 25.4 mm, 1 part

Commit message: Update
Parts:
- removed REF**: Neo-reverse_SMD_4Pin, neo-reverse:Neo-reverse_SMD_4Pin
Changed lines of the file:
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@@
-(kicad_pcb (version 20171130) (host pcbnew 6.0.0-rc1-unknown-efe880b~66~ubuntu16.04.1)
+(kicad_pcb (version 20171130) (host pcbnew 6.0.0-rc1-unknown-efe880b~66~ubuntu18.04.1)
   (general
     (thickness 1.6)
@@
     (tracks 0)
     (zones 0)
-    (modules 1)
+    (modules 0)
     (nets 1)
   )
@@
     (uvia_drill 0.3302)
   )
-  (module neo-reverse:Neo-reverse_SMD_4Pin (layer F.Cu)
-    (at 136.525 94.615)
-    (descr "surface-mounted straight socket strip, 1x04, 2.54mm pitch, single row, style 1 (pin 1 left) (https://cdn.harwin.com/pdfs/M20-786.pdf), script generated")
-    (tags "Surface mounted socket strip SMD 1x04 2.54mm single row style1 pin1 left")
-    (attr smd)
-    (fp_text reference REF** (at 0 -7.62) (layer F.Fab)
-      (effects (font (size 1 1) (thickness 0.15)))
-    )
-    (fp_text value Neo-reverse_SMD_4Pin (at 0 6.985) (layer F.Fab)
-      (effects (font (size 1 1) (thickness 0.15)))
-    )
-    (fp_line (start 4.445 -4.445) (end 4.445 -3.175) (layer F.SilkS) (width 0.15))
-    (fp_line (start 4.445 4.475) (end -4.445 4.445) (layer F.CrtYd) (width 0.05))
-    (fp_line (start -2.175 3.51) (end -2.175 4.11) (layer F.Fab) (width 0.1))
-    (fp_line (start -3.175 3.51) (end -2.175 3.51) (layer F.Fab) (width 0.1))
-    (fp_line (start -2.175 4.11) (end -3.175 4.11) (layer F.Fab) (width 0.1))
-    (fp_line (start -4.445 -4.445) (end 4.445 -4.43) (layer F.CrtYd) (width 0.05))
-    (fp_line (start -4.445 4.445) (end -4.445 -4.445) (layer F.CrtYd) (width 0.05))
-    (fp_text user %R (at 0.635 0 180) (layer F.Fab)
-      (effects (font (size 1 1) (thickness 0.15)))
-    )
-    (fp_line (start 4.445 -4.43) (end 4.445 4.475) (layer F.CrtYd) (width 0.05))
-    (fp_line (start 2.175 -3.51) (end 2.175 -4.11) (layer F.Fab) (width 0.1))
-    (fp_line (start 3.175 -3.51) (end 2.175 -3.51) (layer F.Fab) (width 0.1))
-    (fp_line (start 2.175 -4.11) (end 3.175 -4.11) (layer F.Fab) (width 0.1))
-    (pad 3 smd rect (at -2.795 -3.81 180) (size 1.9 1) (layers F.Cu F.Paste F.Mask))
-    (pad 4 smd rect (at -2.795 3.81 180) (size 1.9 1) (layers F.Cu F.Paste F.Mask))
-    (pad 2 smd rect (at 2.795 3.81) (size 1.9 1) (layers F.Cu F.Paste F.Mask))
-    (pad 1 smd rect (at 2.795 -3.81) (size 1.9 1) (layers F.Cu F.Paste F.Mask))
-    (model ${KIPRJMOD}/vrml/ws2812b_reverse.wrl
-      (at (xyz 0 0 0))
-      (scale (xyz 0.3937 0.3937 0.3937))
-      (rotate (xyz 0 0 0))
-    )
-  )
   (gr_line (start 120.65 82.55) (end 120.65 107.95) (layer Edge.Cuts) (width 0.1524))

Commit message: Update
Parts:
- added U1: NeoReverse-Neo_Reverse, neo-reverse:Neo-reverse_SMD_4Pin, F.Cu at (137.2, 95.5)
Changed lines of the file:
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@@
-(kicad_pcb (version 20171130) (host pcbnew 6.0.0-rc1-unknown-efe880b~66~ubuntu18.04.1)
+(kicad_pcb (version 20171130) (host pcbnew 6.0.0-rc1-unknown-ebdc383~66~ubuntu16.04.1)
   (general
     (thickness 1.6)
@@
     (tracks 0)
     (zones 0)
-    (modules 0)
+    (modules 1)
     (nets 1)
   )
@@
     (pad_to_paste_clearance -0.0762)
     (aux_axis_origin 0 0)
-    (visible_elements FFFEDF7D)
+    (visible_elements FFFFDF7D)
     (pcbplotparams
       (layerselection 0x310fc_80000001)
@@
     (uvia_drill 0.3302)
   )
+  (module neo-reverse:Neo-reverse_SMD_4Pin (layer F.Cu)
+    (at 137.16 95.504)
+    (descr "surface-mounted straight pin header, 1x04, 2.54mm pitch, single row, style 1 (pin 1 left)")
+    (tags "Surface mounted pin header SMD 1x04 2.54mm single row style1 pin1 left")
+    (attr smd)
+    (fp_text reference U1 (at 0 -8.89) (layer F.Fab)
+      (effects (font (size 1 1) (thickness 0.15)))
+    )
+    (fp_text value NeoReverse-Neo_Reverse (at 0 6.985) (layer F.Fab)
+      (effects (font (size 1 1) (thickness 0.15)))
+    )
+    (fp_line (start 3.175 -4.13) (end 1.905 -4.13) (layer F.Fab) (width 0.1))
+    (fp_line (start 1.905 -4.13) (end 1.905 -3.49) (layer F.Fab) (width 0.1))
+    (fp_line (start 1.905 -3.49) (end 3.175 -3.49) (layer F.Fab) (width 0.1))
+    (fp_line (start 5.715 3.49) (end 6.985 3.49) (layer F.Fab) (width 0.1))
+    (fp_line (start 6.985 3.49) (end 6.985 4.13) (layer F.Fab) (width 0.1))
+    (fp_line (start 6.985 4.13) (end 5.715 4.13) (layer F.Fab) (width 0.1))
+    (fp_line (start 8.255 3.175) (end 8.255 4.38) (layer F.SilkS) (width 0.12))
+    (fp_text user %R (at 0 -6.35 180) (layer F.Fab)
+      (effects (font (size 1 1) (thickness 0.15)))
+    )
+    (fp_line (start 8.255 5.08) (end 8.255 -5.08) (layer F.Fab) (width 0.15))
+    (fp_line (start 8.255 -5.08) (end -8.255 -5.08) (layer F.Fab) (width 0.15))
+    (fp_line (start -8.255 -5.08) (end -8.255 5.08) (layer F.Fab) (width 0.15))
+    (fp_line (start -8.255 5.08) (end 8.255 5.08) (layer F.Fab) (width 0.15))
+    (fp_circle (center 0 0) (end 2.5 0) (layer F.Fab) (width 0.15))
+    (pad 4 smd rect (at 2.79 -3.81) (size 2.51 1) (layers F.Cu F.Paste F.Mask))
+    (pad 3 smd rect (at 6.1 3.81) (size 2.51 1) (layers F.Cu F.Paste F.Mask))
+    (pad 1 smd rect (at -6.07 -3.81) (size 2.51 1) (layers F.Cu F.Paste F.Mask))
+    (pad 2 smd rect (at -2.76 3.81) (size 2.51 1) (layers F.Cu F.Paste F.Mask))
+    (model ${KIPRJMOD}/vrml/ws2812b_reverse.wrl
+      (offset (xyz -0.6 0 2.48))
+      (scale (xyz 1 1 1))
+      (rotate (xyz 0 -180 -90))
+    )
+    (model ${KIPRJMOD}/3dShapes/Neo-Reverse-4-Pin.wrl
+      (offset (xyz -4.4 0 0))
+      (scale (xyz 0.3937 0.3937 0.3937))
+      (rotate (xyz 0 0 0))
+    )
+    (model ${KIPRJMOD}/3dShapes/Neo-Reverse-4-Pin.wrl
+      (offset (xyz 4.4 0 0))
+      (scale (xyz 0.3937 0.3937 0.3937))
+      (rotate (xyz 0 0 0))
+    )
+  )
   (gr_line (start 120.65 82.55) (end 120.65 107.95) (layer Edge.Cuts) (width 0.1524))

Commit message: Update
Parts:
- added REF**: Neo-reverse_Mask, neo-reverse:Neo-reverse_Mask, B.Cu at (137.2, 95.5)
- added REF**: Neo-reverse_Mask, neo-reverse:Neo-reverse_Mask, F.Cu at (137.2, 95.5)
Changed lines of the file:
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@@
-(kicad_pcb (version 20171130) (host pcbnew 6.0.0-rc1-unknown-ebdc383~66~ubuntu16.04.1)
+(kicad_pcb (version 20171130) (host pcbnew 6.0.0-rc1-unknown-ebdc383~66~ubuntu18.04.1)
   (general
     (thickness 1.6)
@@
     (tracks 0)
     (zones 0)
-    (modules 1)
+    (modules 3)
     (nets 1)
   )
@@
     (uvia_drill 0.3302)
   )
+  (module neo-reverse:Neo-reverse_Mask (layer B.Cu)
+    (at 137.1854 95.5294 180)
+    (fp_text reference REF** (at 0 3.81 180) (layer B.Fab)
+      (effects (font (size 1 1) (thickness 0.15)) (justify mirror))
+    )
+    (fp_text value Neo-reverse_Mask (at 0 -3.81 180) (layer B.Fab)
+      (effects (font (size 1 1) (thickness 0.15)) (justify mirror))
+    )
+    (pad "" connect circle (at 0 0 180) (size 5 5) (layers B.Mask))
+  )
+  (module neo-reverse:Neo-reverse_Mask (layer F.Cu)
+    (at 137.1854 95.5294)
+    (fp_text reference REF** (at 0 -3.81) (layer F.Fab)
+      (effects (font (size 1 1) (thickness 0.15)))
+    )
+    (fp_text value Neo-reverse_Mask (at 0 3.81) (layer F.Fab)
+      (effects (font (size 1 1) (thickness 0.15)))
+    )
+    (pad "" connect circle (at 0 0) (size 5 5) (layers F.Mask))
+  )
   (module neo-reverse:Neo-reverse_SMD_4Pin (layer F.Cu)
