File: ws2812b_reverse/02/ws2812b_reverse.sch (KiCad schematic (older format))
At the start: 4 parts, among them J1 CONN_01X02, J2 CONN_01X02

Commit message: Add Updates Neo Reverse
Parts:
- removed J1, J2: CONN_01X02, neo-reverse:Pin_half-02x02_P2.54mm, symbol conn:CONN_01X02
- added J1, J2: CONN_01X04, Connector_PinSocket_2.54mm:PinSocket_1x04_P2.54mm_WeMos, symbol conn:CONN_01X04
Connections:
- net GND: now also J2.3 (P3), J2.4 (P4)
- net VCC: now also J1.1 (P1), J1.2 (P2)
- net at LED1.2 (DI): now also J1.3 (P3), J1.4 (P4)
- net at LED1.4 (DO): now also J2.1 (P1), J2.2 (P2)
Changed lines of the file:
@@
 EESchema Schematic File Version 4
 LIBS:ws2812b_reverse-cache
-EELAYER 26 0
+EELAYER 29 0
 EELAYER END
 $Descr USLetter 11000 8500
@@
 Comment4 ""
 $EndDescr
-$Comp
-L conn:CONN_01X02 J1
-U 1 1 5C103029
-P 3950 3950
-F 0 "J1" H 4050 3975 50  0000 L CNN
-F 1 "CONN_01X02" H 4050 3900 50  0000 L CNN
-F 2 "neo-reverse:Pin_half-02x02_P2.54mm" H 3950 3950 50  0001 C CNN
-F 3 "" H 3950 3950 50  0001 C CNN
-	1    3950 3950
-	-1   0    0    -1
-$EndComp
-$Comp
-L conn:CONN_01X02 J2
-U 1 1 5C106126
-P 6100 3925
-F 0 "J2" H 6200 3950 50  0000 L CNN
-F 1 "CONN_01X02" H 6200 3875 50  0000 L CNN
-F 2 "neo-reverse:Pin_half-02x02_P2.54mm" H 6100 3925 50  0001 C CNN
-F 3 "" H 6100 3925 50  0001 C CNN
-	1    6100 3925
-	1    0    0    -1
-$EndComp
 Wire Wire Line
 	4800 4150 4800 4000
@@
 	5800 4150 5800 3875
 Wire Wire Line
-	5800 3875 5900 3875
-Wire Wire Line
-	5900 4400 5900 3975
+	5900 4400 5900 4075
 $Comp
 L power:PWR_FLAG #FLG01
@@
 Connection ~ 4275 3900
 Wire Wire Line
-	4275 3900 4150 3900
-Wire Wire Line
-	4150 4000 4800 4000
+	4275 3900 4200 3900
+Wire Wire Line
+	4150 4000 4200 4000
 Connection ~ 5625 4400
 Wire Wire Line
@@
 Wire Wire Line
 	4575 3600 4575 3500
+$Comp
+L conn:CONN_01X04 J2
+U 1 1 5C48BCA6
+P 6150 3925
+F 0 "J2" H 6228 3966 50  0000 L CNN
+F 1 "CONN_01X04" H 6228 3875 50  0000 L CNN
+F 2 "Connector_PinSocket_2.54mm:PinSocket_1x04_P2.54mm_WeMos" H 6150 3925 50  0001 C CNN
+F 3 "" H 6150 3925 50  0001 C CNN
+	1    6150 3925
+	1    0    0    -1
+$EndComp
+$Comp
+L conn:CONN_01X04 J1
+U 1 1 5C48DB49
+P 3950 3950
+F 0 "J1" H 3867 4315 50  0000 C CNN
+F 1 "CONN_01X04" H 3867 4224 50  0000 C CNN
+F 2 "Connector_PinSocket_2.54mm:PinSocket_1x04_P2.54mm_WeMos" H 3950 3950 50  0001 C CNN
+F 3 "" H 3950 3950 50  0001 C CNN
+	1    3950 3950
+	-1   0    0    -1
+$EndComp
+Wire Wire Line
+	5800 3875 5950 3875
+Wire Wire Line
+	5950 3975 5900 3975
+Wire Wire Line
+	5950 3775 5800 3775
+Wire Wire Line
+	5800 3775 5800 3875
+Connection ~ 5800 3875
+Wire Wire Line
+	5950 4075 5900 4075
+Connection ~ 5900 4075
+Wire Wire Line
+	5900 4075 5900 3975
+Wire Wire Line
+	4150 3800 4200 3800
+Wire Wire Line
+	4200 3800 4200 3900
+Connection ~ 4200 3900
+Wire Wire Line
+	4200 3900 4150 3900
+Wire Wire Line
+	4150 4100 4200 4100
+Wire Wire Line
+	4200 4100 4200 4000
+Connection ~ 4200 4000
+Wire Wire Line
+	4200 4000 4800 4000
 $EndSCHEMATC

Commit message: Update
Parts:
- removed J1, J2: CONN_01X04, Connector_PinSocket_2.54mm:PinSocket_1x04_P2.54mm_WeMos, symbol conn:CONN_01X04
- added J1, J2: Conn_01x02_Female, neo-reverse:Neo-reverser-PinSocket_1x2_P2.54mm, symbol Connector:Conn_01x02_Female
- C1: footprint Capacitor_SMD:C_1206_3216Metric_Pad1.39x1.80mm_HandSolder -> Capacitor_SMD:C_0805_2012Metric_Pad1.15x1.40mm_HandSolder
- LED1: symbol wickerlib:LED-RGB-WS2812B-4SMD -> ws2812b_reverse-rescue:LED-RGB-WS2812B-4SMD-wickerlib
Connections:
- net GND: now also J2.2 (Pin_2)
- net VCC: now also J1.1 (Pin_1)
- net at LED1.2 (DI): now also J1.2 (Pin_2)
- net at LED1.4 (DO): now also J2.1 (Pin_1)
Changed lines of the file:
@@
 Wire Wire Line
 	5800 4150 5800 3875
-Wire Wire Line
-	5900 4400 5900 4075
 $Comp
 L power:PWR_FLAG #FLG01
@@
 F 0 "C1" V 4323 3750 50  0000 C CNN
 F 1 "C" H 4725 3750 50  0000 C CNN
-F 2 "Capacitor_SMD:C_1206_3216Metric_Pad1.39x1.80mm_HandSolder" H 4613 3600 50  0001 C CNN
+F 2 "Capacitor_SMD:C_0805_2012Metric_Pad1.15x1.40mm_HandSolder" H 4613 3600 50  0001 C CNN
 F 3 "" H 4575 3750 50  0000 C CNN
 	1    4575 3750
@@
 Connection ~ 4575 3900
 Connection ~ 4275 3900
-Wire Wire Line
-	4275 3900 4200 3900
-Wire Wire Line
-	4150 4000 4200 4000
 Connection ~ 5625 4400
 Wire Wire Line
 	5625 4400 5900 4400
 $Comp
-L wickerlib:LED-RGB-WS2812B-4SMD LED1
+L ws2812b_reverse-rescue:LED-RGB-WS2812B-4SMD-wickerlib LED1
 U 1 1 5C1015C7
 P 5250 3900
@@
 Wire Wire Line
 	4575 3600 4575 3500
-$Comp
-L conn:CONN_01X04 J2
-U 1 1 5C48BCA6
-P 6150 3925
-F 0 "J2" H 6228 3966 50  0000 L CNN
-F 1 "CONN_01X04" H 6228 3875 50  0000 L CNN
-F 2 "Connector_PinSocket_2.54mm:PinSocket_1x04_P2.54mm_WeMos" H 6150 3925 50  0001 C CNN
-F 3 "" H 6150 3925 50  0001 C CNN
-	1    6150 3925
-	1    0    0    -1
-$EndComp
-$Comp
-L conn:CONN_01X04 J1
-U 1 1 5C48DB49
-P 3950 3950
-F 0 "J1" H 3867 4315 50  0000 C CNN
-F 1 "CONN_01X04" H 3867 4224 50  0000 C CNN
-F 2 "Connector_PinSocket_2.54mm:PinSocket_1x04_P2.54mm_WeMos" H 3950 3950 50  0001 C CNN
-F 3 "" H 3950 3950 50  0001 C CNN
-	1    3950 3950
-	-1   0    0    -1
-$EndComp
 Wire Wire Line
 	5800 3875 5950 3875
 Wire Wire Line
 	5950 3975 5900 3975
+$Comp
+L Connector:Conn_01x02_Female J2
+U 1 1 5C4A65E0
+P 6150 3875
+F 0 "J2" H 6178 3805 50  0000 L CNN
+F 1 "Conn_01x02_Female" H 6178 3760 50  0001 L CNN
+F 2 "neo-reverse:Neo-reverser-PinSocket_1x2_P2.54mm" H 6150 3875 50  0001 C CNN
+F 3 "~" H 6150 3875 50  0001 C CNN
+	1    6150 3875
+	1    0    0    -1
+$EndComp
+$Comp
+L Connector:Conn_01x02_Female J1
+U 1 1 5C4A7F1A
+P 3950 3900
+F 0 "J1" H 3842 4085 50  0000 C CNN
+F 1 "Conn_01x02_Female" H 4400 4025 50  0001 C CNN
+F 2 "neo-reverse:Neo-reverser-PinSocket_1x2_P2.54mm" H 3950 3900 50  0001 C CNN
+F 3 "~" H 3950 3900 50  0001 C CNN
+	1    3950 3900
+	-1   0    0    -1
+$EndComp
 Wire Wire Line
-	5950 3775 5800 3775
+	5900 3975 5900 4400
 Wire Wire Line
-	5800 3775 5800 3875
-Connection ~ 5800 3875
+	4150 3900 4275 3900
 Wire Wire Line
-	5950 4075 5900 4075
-Connection ~ 5900 4075
-Wire Wire Line
-	5900 4075 5900 3975
-Wire Wire Line
-	4150 3800 4200 3800
-Wire Wire Line
-	4200 3800 4200 3900
-Connection ~ 4200 3900
-Wire Wire Line
-	4200 3900 4150 3900
-Wire Wire Line
-	4150 4100 4200 4100
-Wire Wire Line
-	4200 4100 4200 4000
-Connection ~ 4200 4000
-Wire Wire Line
-	4200 4000 4800 4000
+	4150 4000 4800 4000
 $EndSCHEMATC
