File: tft-shield/001/001.sch (KiCad schematic (older format))
At the start: 7 parts, among them J1 CONN_01X08, Q1 S8050, U1 TFT_0.9680*160

Commit message: Add some changess & 3d model
Parts:
- C1: footprint Capacitor_SMD:C_1206_3216Metric_Pad1.42x1.75mm_HandSolder -> Capacitor_SMD:C_0805_2012Metric_Pad1.15x1.40mm_HandSolder
- R1, R2, R3: footprint Resistor_SMD:R_1206_3216Metric_Pad1.39x1.80mm_HandSolder -> Resistor_SMD:R_0805_2012Metric_Pad1.15x1.40mm_HandSolder
Changed lines of the file:
@@
 F 0 "R1" V 7404 3675 50  0000 C CNN
 F 1 "1k" V 7495 3675 50  0000 C CNN
-F 2 "Resistor_SMD:R_1206_3216Metric_Pad1.39x1.80mm_HandSolder" H 7600 3675 50  0001 C CNN
+F 2 "Resistor_SMD:R_0805_2012Metric_Pad1.15x1.40mm_HandSolder" H 7600 3675 50  0001 C CNN
 F 3 "" H 7600 3675 50  0001 C CNN
 	1    7600 3675
@@
 F 0 "R3" V 8279 3350 50  0000 C CNN
 F 1 "10ohm" V 8370 3350 50  0000 C CNN
-F 2 "Resistor_SMD:R_1206_3216Metric_Pad1.39x1.80mm_HandSolder" H 8475 3350 50  0001 C CNN
+F 2 "Resistor_SMD:R_0805_2012Metric_Pad1.15x1.40mm_HandSolder" H 8475 3350 50  0001 C CNN
 F 3 "" H 8475 3350 50  0001 C CNN
 	1    8475 3350
@@
 F 0 "R2" H 7884 3946 50  0000 L CNN
 F 1 "10k" H 7884 3855 50  0000 L CNN
-F 2 "Resistor_SMD:R_1206_3216Metric_Pad1.39x1.80mm_HandSolder" H 7825 3900 50  0001 C CNN
+F 2 "Resistor_SMD:R_0805_2012Metric_Pad1.15x1.40mm_HandSolder" H 7825 3900 50  0001 C CNN
 F 3 "" H 7825 3900 50  0001 C CNN
 	1    7825 3900
@@
 F 0 "C1" V 4350 3950 50  0000 C CNN
 F 1 "1uF" V 4350 4150 50  0000 C CNN
-F 2 "Capacitor_SMD:C_1206_3216Metric_Pad1.42x1.75mm_HandSolder" H 4400 4050 50  0001 C CNN
+F 2 "Capacitor_SMD:C_0805_2012Metric_Pad1.15x1.40mm_HandSolder" H 4400 4050 50  0001 C CNN
 F 3 "" H 4400 4050 50  0001 C CNN
 	1    4400 4050
