File: Bast_Shield/003/Bast-Pro-Mini-M0.kicad_pcb (KiCad board)
At the start: 2 copper layers, 21.6 x 31.8 mm, 8 parts, among them P1 Digital, P3 Analog, Q1 S8050, U1 TFT_0.9680*160

Commit message: Various updates
Parts:
- added svg2mod: G***, tft-shield:Bast_5, B.Cu at (154.7, 98.7)
- added svg2mod: G***, tft-shield:firma, F.Cu at (145.8, 90.8)
- moved U1 0.51 mm to (145.5, 98.4)
Other:
- board text added: "Designed by"
