File: Hackster/Hackster_Round/001.kicad_pcb (KiCad board)
At the start: 2 copper layers, 74.7 x 96.8 mm, 69 parts, among them J1 CONN_01X02, J10 TEST_1P, J11 TEST_1P, J12 TEST_1P, J13 TEST_1P, J14 TEST_1P, J15 TEST_1P, J16 TEST_1P, J17 GS2, J2 TEST_1P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

Commit message: Add KiCad Template
Parts:
- removed B-G***: B-LOGO, varios:bricolabs-14
- removed Eyes***: LOGO, Mazmaker:Oshwdem_Eyes_08
- removed G***: LOGO, varios:OSHpark-2-1800
- removed G***Ki: Ki-LOGO, varios:Ki-2500
- removed GBSilk***: LOGO, varios:greynaga6-2
- removed GS***: v, varios:greynaga6-2-cooper
- removed Head***: LOGO, Mazmaker:Oshwdem_Head_01
- removed Mouth***: LOGO, Mazmaker:Oshwdem_Mouth_01
- removed PP-G***: PP-LOGO, varios:OSHpark-1-1200
- removed PPP-G***: PPP-LOGO, varios:OSHpark-1-2000
- removed PPPP-G***: PPPP-LOGO, varios:OSHpark-2-1800
- removed REF**: MountingHole_3.2mm_M3_DIN965_Pad, Mazmaker:MountingHole_3.2mm_M3_DIN965_Pad
- removed REF***: OSHW-Logo2_7.3x6mm_SilkScreen, Symbols:OSHW-Logo2_7.3x6mm_SilkScreen
- removed REF1**, REF10**, REF11**, REF12**, REF13**, REF14**, REF15**, REF16**, REF2**, REF3**, REF4**, REF5**, REF6**, REF7**, REF8**, REF9**: PADS, Mazmaker:PADS
- removed p-G***: P-LOGO, varios:OSHpark-1-1000
- C1, C2, C3, C4: footprint Capacitors_SMD:C_0805_HandSoldering -> Hackster_Round:C_0805_HandSoldering; moved to F.Cu
- D1: footprint OSHwi:D_SOD-123 -> Hackster_Round:D_SOD-123; moved to F.Cu
- D2: footprint OSHwi:LED_0805 -> Hackster_Round:LED_0805
- J1: footprint Connectors_Molex:Molex_PicoBlade_53261-0271_02x1.25mm_Angled -> Hackster_Round:Molex_PicoBlade_53261-0271_02x1.25mm_Angled; moved to F.Cu
- J10, J11, J12, J13, J14, J15, J16, J2, J3, J4, J5, J6, J7, J8, J9: footprint Wickerlib:CONN-HEADER-STRAIGHT-P2.54MM-1x01 -> Hackster_Round:CONN-HEADER-STRAIGHT-P2.54MM-1x01
- J17: footprint Connectors:GS2 -> Hackster_Round:GS2; moved to F.Cu
- LED1, LED2, LED3, LED4, LED5: footprint OSHwi:WS2812B -> Hackster_Round:WS2812B
- R1, R2, R3, R4, R5, R6, R7: footprint Resistors_SMD:R_0805_HandSoldering -> Hackster_Round:R_0805_HandSoldering; moved to F.Cu
- SW1, SW2: footprint Buttons_Switches_SMD:SW_SPST_B3U-1000P -> Hackster_Round:SW_SPST_B3U-1000P
- U1: footprint ESP8266:ESP-12S_SMD -> Hackster_Round:ESP-12S_SMD; moved to F.Cu
- U2: footprint TO_SOT_Packages_SMD:SOT-23-5_HandSoldering -> Hackster_Round:SOT-23-5_HandSoldering; moved to F.Cu
- moved J13 61.1 mm to (174.2, 91.7)
- moved J15 57.7 mm to (172.1, 103.9)
- moved LED5 56.6 mm to (167.2, 87.4)
- moved R6 56.2 mm to (174.4, 85.4), turned to 0 degrees
- moved J16 55.9 mm to (162.9, 112.0)
- moved R3 54.1 mm to (155.1, 103.8), turned to 0 degrees
- moved LED4 53.4 mm to (156.5, 95.5), turned to 0 degrees
- moved R7 52.3 mm to (163.7, 92.4), turned to 0 degrees
- moved LED3 52.1 mm to (147.8, 102.5), turned to 0 degrees
- moved J3 48.5 mm to (168.1, 102.8)
- moved J5 47.8 mm to (165.2, 107.9)
- moved J9 44.4 mm to (160.0, 103.9)
- moved J11 41.2 mm to (157.1, 107.9)
- moved R1 40.8 mm to (144.3, 112.1), turned to 0 degrees
- moved J7 40.0 mm to (154.7, 112.0)
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Routing:
- net +3.3V: track 161.8 -> 0.00 mm, vias 3 -> 0
- net GPIO16: track 53.3 -> 0.00 mm, vias 3 -> 0
- net GPIO0: track 50.8 -> 0.00 mm, vias 1 -> 0
- net REST: track 47.1 -> 0.00 mm, vias 3 -> 0
- net GPIO15: track 45.0 -> 0.00 mm, vias 1 -> 0
- net GPIO14: track 43.5 -> 0.00 mm, vias 2 -> 0
- net ADC: track 41.7 -> 0.00 mm, vias 2 -> 0
- net GPIO12: track 40.1 -> 0.00 mm, vias 2 -> 0
- net CH_PD: track 40.0 -> 0.00 mm, vias 3 -> 0
- net GPIO2: track 38.7 -> 0.00 mm, vias 1 -> 0
- net GPIO13: track 37.9 -> 0.00 mm, vias 1 -> 0
- net GPIO5: track 33.2 -> 0.00 mm, vias 1 -> 0
- net GPIO4: track 32.9 -> 0.00 mm, vias 4 -> 0
- net RXD: track 31.8 -> 0.00 mm, vias 1 -> 0
- net TXD: track 25.6 -> 0.00 mm, vias 1 -> 0
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- removed copper zone on B.Cu, net GND
- removed copper zone on F.Cu, net GND
Other:
- board outline removed
- board text removed: "+"
- board text removed: "-"
- board text removed: "0"
- board text removed: "12"
- board text removed: "13"
- board text removed: "14"
- board text removed: "15"
- board text removed: "16"
- board text removed: "4"
- board text removed: "5"
- board text removed: "ADC"
- board text removed: "CH_PD"
- board text removed: "DSJ"
- board text removed: "Designed by"
- board text removed: "GND"
- board text removed: "ON"
- board text removed: "RESET"
- board text removed: "RST"
- board text removed: "RX"
- board text removed: "TX"
- board text removed: "USER/FLASH"
- board text removed: "VIN"
