File: Escornabot/CPU/001/Escorna_CPU_1_20.kicad_pcb (KiCad board)
At the start: 2 copper layers, 50 x 50 mm, 41 parts, among them IC1 ULN2803, U2 ESP01, U3 MA04-1, U6 1117-3.3, X1.1 AK550_2

Commit message: Updates
Other:
- board text removed: "CC BY-SA 4.0"
Changed lines of the file:
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@@
-(kicad_pcb (version 20171130) (host pcbnew 6.0.0-rc1-unknown-55b5c71~66~ubuntu16.04.1)
+(kicad_pcb (version 20171130) (host pcbnew 5.1.0-rc1-unknown-ec59361f~76~ubuntu18.04.1)
   (general
     (thickness 1.6)
-    (drawings 76)
+    (drawings 75)
     (tracks 304)
     (zones 0)
@@
     (effects (font (size 1.35128 1.35128) (thickness 0.113792)) (justify right top))
   )
-  (gr_text "CC BY-SA 4.0" (at 147.3926 102.6141 90) (layer F.SilkS)
-    (effects (font (size 0.76 0.76) (thickness 0.064)) (justify right top))
-  )
   (gr_text BlueT (at 160.5956 88.1941) (layer F.SilkS)

Commit message: update
Routing:
- net /RST: track 25.2 -> 34.0 mm
- net Net-(R5-Pad2): track 17.1 -> 16.1 mm
- net (no net): vias 0 -> 18
