File: Escorni_Badge/001/001.sch (KiCad schematic (older format))
At the start: 1 part

Commit message: Update Escorni
Parts:
- removed R1: R, Resistor_SMD:R_1206_3216Metric_Pad1.39x1.80mm_HandSolder, symbol device:R
- added C1, C2: 4.7uF, 001:C_1206_HandSoldering, symbol Device:C
- added C3: 22nF, 001:C_1206_HandSoldering, symbol Device:C
- added CAP1: Escorni_Touch, 001:escorni-Touch_02_100mm, symbol Escorni_Badge:Escorni_Touch
- added D1: MBRA140, 001:DIODE-SMA, symbol wickerlib:DIODE-SCHOTTKY-40V-1A-MBRA140-SMA
- added D2: ON, 001:LED_1206_HandSoldering, symbol 001-rescue:LED-RESCUE-001-001-rescue-HG_002-rescue
- added J1: CONN_01X02, 001:Pin_Header_Straight_1x02_Pitch2.54mm_SMD_Pin1Left, symbol 001-rescue:CONN_01X02-conn
- added J2: CONN_01X02, Connector_JST:JST_PH_S2B-PH-SM4-TB_1x02-1MP_P2.00mm_Horizontal, symbol 001-rescue:CONN_01X02-conn
- added J3: CONN_02X03, 001:Pin_Header_Straight_2x03_Pitch2.54mm_SMD, symbol 001-rescue:CONN_02X03-conn
- added J4: CONN_01X03, 001:Pin_Header_Straight_1x03_Pitch2.54mm_SMD_Pin1Left, symbol 001-rescue:CONN_01X03-conn
- added J5: CONN_01X03, 001:Pin_Header_Straight_1x03_Pitch2.54mm_SMD_Pin1Right, symbol 001-rescue:CONN_01X03-conn
- added LED1, LED2, LED3, LED4, LED5: WS2812B, 001:WS2812B, symbol wickerlib:LED-RGB-WS2812B-4SMD
- added R1: 1Mohm, 001:R_1206_HandSoldering, symbol Device:R
- added R2: 1k, 001:R_1206_HandSoldering, symbol pspice:R
- added S1: MSK12C02_SWITCH-SLIDE-SPDT, 001:MSK12C02, symbol wickerlib:SWITCH-SLIDE-SPDT-100MA-12V
- added SilKs1: Escorni_Art, 001:escorni-badge-new_02_100mm, symbol 001-rescue:HG_SilKs_2-HG
- added U1: LM340MP-5.0/NOPB, Package_TO_SOT_SMD:SOT-223-3_TabPin2, symbol 001-rescue:LM7805_TO220-regul
- added U2: ATTINY85-20SU, Package_SO:SOIJ-8_5.3x5.3mm_P1.27mm, symbol 001-rescue:ATTINY85-20SU-atmel
Connections:
- net labels added: +5V, 3-A3, 4-A2, MISO-1-PWM, MOSI-0-PWM, RESET, SCK-2-A1, VBAT, VCC
- net labels removed: +3.3V
- wire segments 0 -> 64
- no-connect marks 0 -> 2
Other:
- note added: "ATTINY 85"
- note added: "Agregar una conexión manual a la H"
- note added: "CAPACITIVE SENSOR"
- note added: "Escornabot Art"
- note added: "ISCP"
- note added: "NEOPIXELS"
- note added: "POWER & FILTERING"
- note added: "POWER LED"
- note added: "PROGRAMING PORT & I/O PINS"
- note added: "USER PINS"
