File: MazBasica/Maz-ONE-0/Arduino_As_Uno.kicad_pcb (KiCad board)
At the start: 2 copper layers, 48.3 x 53.3 mm, 23 parts, among them J1 CONN_01X04, J2 CONN_01X03, J3 CONN_01X03, J4 CONN_01X06, J5 CONN_01X01, P1 Power, P2 Analog, P3 Digital, P4 Digital, SW1 SW_Push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

Commit message: Add Maz-ONE
Parts:
- removed J5: CONN_01X01, Connector_PinHeader_2.54mm:PinHeader_1x01_P2.54mm_Vertical
- added P5: TFT Port, Maz-ONE:Socket_Strip_Arduino_1x08, F.Cu at (114.8, 80.6)
- R6: value 2k -> 2k2
- moved BZ1 7.62 mm to (144.0, 88.3), turned to 180 degrees
- moved RV1 0.64 mm to (147.8, 117.5)
- renumbered LDR to R1
Connections:
- J1 pad 3: (no net) -> Net-(J1-Pad3)
- J4 pad 1: (no net) -> Net-(J4-Pad1)
- J4 pad 6: (no net) -> Net-(J4-Pad6)
- LED3 pad 4: (no net) -> Net-(LED3-Pad4)
- P1 pad 1: (no net) -> Net-(P1-Pad1)
- P1 pad 2: (no net) -> /IOREF
- P1 pad 4: (no net) -> +3V3
- P1 pad 8: (no net) -> /Vin
- P3 pad 10: (no net) -> /8
- P3 pad 3: (no net) -> /AREF
- P3 pad 5: (no net) -> /13(SCK)
- P3 pad 6: (no net) -> /12(MISO)
- P3 pad 7: (no net) -> /11(**/MOSI)
- P3 pad 8: (no net) -> /10(**/SS)
- P4 pad 1: (no net) -> /7
- P4 pad 4: (no net) -> /4
Routing:
- added copper zone on B.Cu, net GND
- added copper zone on F.Cu, net GND
Other:
- board text added: "Maz-ONE"
- board text removed: "MAZ-ONE"
