File: Escorni_Badge/002/001.sch (KiCad schematic (older format))
At the start: 22 parts, among them J1 CONN_01X02, J2 CONN_01X02, J3 CONN_02X03, J4 CONN_01X03, J5 CONN_01X03, U1 LM340MP-5.0/NOPB, U2 ATTINY85-20SU

Commit message: Escorni NANO update
Parts:
- C1, C2, C3: footprint 001:C_1206_HandSoldering -> 002:C_1206_HandSoldering
- CAP1: footprint 001:escorni-Touch_02_100mm -> 002:escorni-Touch_02_100mm
- D1: footprint 001:DIODE-SMA -> 002:DIODE-SMA; symbol wickerlib:DIODE-SCHOTTKY-40V-1A-MBRA140-SMA -> 001-rescue:DIODE-SCHOTTKY-40V-1A-MBRA140-SMA-wickerlib
- D2: footprint 001:LED_1206_HandSoldering -> 002:LED_1206_HandSoldering
- J1: footprint 001:Pin_Header_Straight_1x02_Pitch2.54mm_SMD_Pin1Left -> 002:Pin_Header_Straight_1x02_Pitch2.54mm_SMD_Pin1Left
- J4: footprint 001:Pin_Header_Straight_1x03_Pitch2.54mm_SMD_Pin1Left -> 002:Pin_Header_Straight_1x03_Pitch2.54mm_SMD_Pin1Left
- J5: footprint 001:Pin_Header_Straight_1x03_Pitch2.54mm_SMD_Pin1Right -> 002:Pin_Header_Straight_1x03_Pitch2.54mm_SMD_Pin1Right
- LED1, LED2, LED3, LED4, LED5: footprint 001:WS2812B -> 002:WS2812B; symbol wickerlib:LED-RGB-WS2812B-4SMD -> 001-rescue:LED-RGB-WS2812B-4SMD-wickerlib
- R1: footprint 001:R_1206_HandSoldering -> 002:R_1206_HandSoldering
- S1: footprint 001:MSK12C02 -> 002:MSK12C02; symbol wickerlib:SWITCH-SLIDE-SPDT-100MA-12V -> 001-rescue:SWITCH-SLIDE-SPDT-100MA-12V-wickerlib
- SilKs1: footprint 001:escorni-badge-new_02_100mm -> 002:escorni-badge-new_03_100mm
Changed lines of the file:
@@
 $EndComp
 $Comp
-L wickerlib:LED-RGB-WS2812B-4SMD LED1
+L 001-rescue:LED-RGB-WS2812B-4SMD-wickerlib LED1
 U 1 1 595D0515
 P 8685 4100
 F 0 "LED1" H 8735 4475 50  0000 C CNN
 F 1 "WS2812B" H 8735 4384 50  0000 C CNN
-F 2 "001:WS2812B" H 8685 3750 50  0001 C CIN
+F 2 "002:WS2812B" H 8685 3750 50  0001 C CIN
 F 3 "http://www.adafruit.com/datasheets/WS2812B.pdf" H 8685 4100 5   0001 C CNN
 F 4 "LED RGB WS2812B W/DVR 4SMD" H 8685 3750 50  0001 C CIN "Description"
@@
 $EndComp
 $Comp
-L wickerlib:LED-RGB-WS2812B-4SMD LED2
+L 001-rescue:LED-RGB-WS2812B-4SMD-wickerlib LED2
 U 1 1 595D08CE
 P 7535 4100
 F 0 "LED2" H 7585 4475 50  0000 C CNN
 F 1 "WS2812B" H 7585 4384 50  0000 C CNN
-F 2 "001:WS2812B" H 7535 3750 50  0001 C CIN
+F 2 "002:WS2812B" H 7535 3750 50  0001 C CIN
 F 3 "http://www.adafruit.com/datasheets/WS2812B.pdf" H 7535 4100 5   0001 C CNN
 F 4 "LED RGB WS2812B W/DVR 4SMD" H 7535 3750 50  0001 C CIN "Description"
@@
 $EndComp
 $Comp
-L wickerlib:LED-RGB-WS2812B-4SMD LED3
+L 001-rescue:LED-RGB-WS2812B-4SMD-wickerlib LED3
 U 1 1 595D1904
 P 6260 4100
 F 0 "LED3" H 6310 4475 50  0000 C CNN
 F 1 "WS2812B" H 6310 4384 50  0000 C CNN
-F 2 "001:WS2812B" H 6260 3750 50  0001 C CIN
+F 2 "002:WS2812B" H 6260 3750 50  0001 C CIN
 F 3 "http://www.adafruit.com/datasheets/WS2812B.pdf" H 6260 4100 5   0001 C CNN
 F 4 "LED RGB WS2812B W/DVR 4SMD" H 6260 3750 50  0001 C CIN "Description"
@@
 $EndComp
 $Comp
-L wickerlib:LED-RGB-WS2812B-4SMD LED4
+L 001-rescue:LED-RGB-WS2812B-4SMD-wickerlib LED4
 U 1 1 595D190F
 P 5010 4100
 F 0 "LED4" H 5060 4475 50  0000 C CNN
 F 1 "WS2812B" H 5060 4384 50  0000 C CNN
-F 2 "001:WS2812B" H 5010 3750 50  0001 C CIN
+F 2 "002:WS2812B" H 5010 3750 50  0001 C CIN
 F 3 "http://www.adafruit.com/datasheets/WS2812B.pdf" H 5010 4100 5   0001 C CNN
 F 4 "LED RGB WS2812B W/DVR 4SMD" H 5010 3750 50  0001 C CIN "Description"
@@
 F 0 "D2" V 2355 7205 50  0000 R CNN
 F 1 "ON" V 2265 7210 50  0000 R CNN
-F 2 "001:LED_1206_HandSoldering" H 2315 7385 50  0001 C CNN
+F 2 "002:LED_1206_HandSoldering" H 2315 7385 50  0001 C CNN
 F 3 "" H 2315 7385 50  0001 C CNN
 	1    2315 7385
@@
 VBAT
 $Comp
-L wickerlib:DIODE-SCHOTTKY-40V-1A-MBRA140-SMA D1
+L 001-rescue:DIODE-SCHOTTKY-40V-1A-MBRA140-SMA-wickerlib D1
 U 1 1 598120B7
 P 6775 1075
 F 0 "D1" H 6707 1075 50  0000 R CNN
 F 1 "MBRA140" H 6707 1120 50  0001 R CNN
-F 2 "001:DIODE-SMA" H 6775 725 50  0001 C CIN
+F 2 "002:DIODE-SMA" H 6775 725 50  0001 C CIN
 F 3 "http://www.vishay.com/docs/94301/vs-mbra140trpbf.pdf" V 6775 1075 10  0001 C CNN
 F 4 "DIODE SCHOTTKY 40V 1A MBRA140 SMA" H 6775 725 50  0001 C CIN "Description"
@@
 F 0 "J1" H 6010 1260 50  0000 C CNN
 F 1 "CONN_01X02" V 6110 1110 50  0000 C CNN
-F 2 "001:Pin_Header_Straight_1x02_Pitch2.54mm_SMD_Pin1Left" H 6010 1110 50  0001 C CNN
+F 2 "002:Pin_Header_Straight_1x02_Pitch2.54mm_SMD_Pin1Left" H 6010 1110 50  0001 C CNN
 F 3 "" H 6010 1110 50  0001 C CNN
 	1    6010 1110
@@
 F 0 "J4" H 2600 6335 50  0000 C CNN
 F 1 "CONN_01X03" V 2700 6135 50  0000 C CNN
-F 2 "001:Pin_Header_Straight_1x03_Pitch2.54mm_SMD_Pin1Left" H 2600 6135 50  0001 C CNN
+F 2 "002:Pin_Header_Straight_1x03_Pitch2.54mm_SMD_Pin1Left" H 2600 6135 50  0001 C CNN
 F 3 "" H 2600 6135 50  0001 C CNN
 	1    2600 6135
@@
 F 0 "J5" H 2980 6335 50  0000 C CNN
 F 1 "CONN_01X03" V 3080 6135 50  0000 C CNN
-F 2 "001:Pin_Header_Straight_1x03_Pitch2.54mm_SMD_Pin1Right" H 2980 6135 50  0001 C CNN
+F 2 "002:Pin_Header_Straight_1x03_Pitch2.54mm_SMD_Pin1Right" H 2980 6135 50  0001 C CNN
 F 3 "" H 2980 6135 50  0001 C CNN
 	1    2980 6135
@@
 F 0 "SilKs1" H 4338 7251 50  0000 L CNN
 F 1 "Escorni_Art" H 4338 7160 50  0000 L CNN
-F 2 "001:escorni-badge-new_02_100mm" H 4160 7205 50  0001 C CNN
+F 2 "002:escorni-badge-new_03_100mm" H 4160 7205 50  0001 C CNN
 F 3 "" H 4160 7205 50  0001 C CNN
 	1    4160 7205
@@
 Agregar una conexión manual a la H
 $Comp
-L wickerlib:SWITCH-SLIDE-SPDT-100MA-12V S1
+L 001-rescue:SWITCH-SLIDE-SPDT-100MA-12V-wickerlib S1
 U 1 1 5BD9DEF7
 P 7055 1175
 F 0 "S1" H 7050 1040 50  0000 C CNN
 F 1 "MSK12C02_SWITCH-SLIDE-SPDT" H 7030 1355 50  0001 C CNN
-F 2 "001:MSK12C02" H 7055 825 50  0001 C CIN
+F 2 "002:MSK12C02" H 7055 825 50  0001 C CIN
 F 3 "https://es.aliexpress.com/item/10pcs-Slide-Switch-On-OFF-2-Position-1P2T-SPDT-Miniature-Horizontal-Slide-Switch-SMD-7-Pin/32770836506.html?spm=a219c.10010108.1000016.1.415e538dUbCoPc&isOrigTitle=true" H 7055 975 5   0001 C CNN
 F 4 "SWITCH SLIDE SPDT" H 7055 825 50  0001 C CIN "Description"
@@
 	7520 1175 7740 1175
 $Comp
-L wickerlib:LED-RGB-WS2812B-4SMD LED5
+L 001-rescue:LED-RGB-WS2812B-4SMD-wickerlib LED5
 U 1 1 595D1F1E
 P 3735 4100
 F 0 "LED5" H 3785 4475 50  0000 C CNN
 F 1 "WS2812B" H 3785 4384 50  0000 C CNN
-F 2 "001:WS2812B" H 3735 3750 50  0001 C CIN
+F 2 "002:WS2812B" H 3735 3750 50  0001 C CIN
 F 3 "http://www.adafruit.com/datasheets/WS2812B.pdf" H 3735 4100 5   0001 C CNN
 	1    3735 4100
@@
 F 0 "R1" V 8250 6175 50  0000 C CNN
 F 1 "1Mohm" V 8450 6175 50  0000 C CNN
-F 2 "001:R_1206_HandSoldering" V 8280 6175 50  0001 C CNN
+F 2 "002:R_1206_HandSoldering" V 8280 6175 50  0001 C CNN
 F 3 "~" H 8350 6175 50  0001 C CNN
 	1    8350 6175
@@
 F 0 "CAP1" H 9159 6103 60  0000 L CNN
 F 1 "Escorni_Touch" H 9159 5997 60  0000 L CNN
-F 2 "001:escorni-Touch_02_100mm" H 8850 6350 60  0001 C CNN
+F 2 "002:escorni-Touch_02_100mm" H 8850 6350 60  0001 C CNN
 F 3 "" H 8925 6050 60  0000 C CNN
 	1    8925 6050
@@
 F 0 "C3" H 9440 5006 50  0000 L CNN
 F 1 "22nF" H 9440 4915 50  0000 L CNN
-F 2 "001:C_1206_HandSoldering" H 9363 4810 50  0001 C CNN
+F 2 "002:C_1206_HandSoldering" H 9363 4810 50  0001 C CNN
 F 3 "~" H 9325 4960 50  0001 C CNN
 	1    9325 4960
@@
 F 0 "C1" H 7420 1571 50  0000 L CNN
 F 1 "4.7uF" H 7420 1480 50  0000 L CNN
-F 2 "001:C_1206_HandSoldering" H 7343 1375 50  0001 C CNN
+F 2 "002:C_1206_HandSoldering" H 7343 1375 50  0001 C CNN
 F 3 "~" H 7305 1525 50  0001 C CNN
 	1    7305 1525
@@
 F 0 "C2" H 9110 1571 50  0000 L CNN
 F 1 "4.7uF" H 9110 1480 50  0000 L CNN
-F 2 "001:C_1206_HandSoldering" H 9033 1375 50  0001 C CNN
+F 2 "002:C_1206_HandSoldering" H 9033 1375 50  0001 C CNN
 F 3 "~" H 8995 1525 50  0001 C CNN
 	1    8995 1525
