File: Regla-Leds/001.sch (KiCad schematic (older format))
At the start: 20 parts, among them J1 CONN_02X03, J2 CONN_01X02, J3 CONN_01X02, SW1 SW_SPDT, U1 ATTINY85-20SU, U2 LM340MP-5.0/NOPB

Commit message: Updates
Parts:
- removed D1: ON, LED_SMD:LED_1206_3216Metric_Pad1.42x1.75mm_HandSolder, symbol 001-rescue:LED-RESCUE-001-001-rescue-HG_002-rescue
- added D9: LED, LED_THT:LED_D5.0mm, symbol Device:LED
- renumbered D2 to D1, D3 to D2, D4 to D3, D5 to D4, D6 to D5, D7 to D6, D8 to D7, D9 to D8
Connections:
- wire segments 45 -> 59
Other:
- note added: "CharliePlex"
- note added: "NeoPixel"
- note removed: "NEOPIXELS"
- moved on the sheet: C1, C2, C3, D1, D10, D2, D3, D4, D5, D6, D7, D8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
