File: Escorni_Badge/002-Nano/NANO33IoTV2.0.sch (KiCad schematic (older format))
At the start: 10 parts, among them J1 Arduino-NANO-33

Commit message: Escorni NANO update
Parts:
- removed D1: ON, 002:LED_1206_HandSoldering, symbol NANO33IoTV2.0-rescue:LED-RESCUE-001-001-rescue-HG_002-rescue-001-rescue
- removed LED1, LED2, LED3, LED4, LED5: WS2812B, 002:WS2812B, symbol wickerlib:LED-RGB-WS2812B-4SMD
- removed R1: 1k, 001:R_1206_HandSoldering, symbol pspice:R
- added D1: LED, LED_SMD:LED_0805_2012Metric_Pad1.15x1.40mm_HandSolder, symbol Device:LED
- added LED1, LED2, LED3, LED4, LED5: WS2812B, 002:WS2812B, symbol NANO33IoTV2.0-rescue:WS2812B
- added R1: 1k, Resistor_SMD:R_0805_2012Metric_Pad1.15x1.40mm_HandSolder, symbol Device:R
- SilKs1: symbol NANO33IoTV2.0-rescue:HG_SilKs_2-HG-001-rescue -> 001-rescue:HG_SilKs_2-HG
Connections:
- net labels added: NEO-D3
- net labels removed: +5V, 4-A2
- wire segments 34 -> 38
Other:
- note added: "?"
- moved on the sheet: C1
Changed lines of the file:
@@
 L power:GND #PWR0101
 U 1 1 595C807D
-P 2210 3175
-F 0 "#PWR0101" H 2210 2925 50  0001 C CNN
-F 1 "GND" H 2215 3002 50  0000 C CNN
-F 2 "" H 2210 3175 50  0001 C CNN
-F 3 "" H 2210 3175 50  0001 C CNN
-	1    2210 3175
-	1    0    0    -1
-$EndComp
-$Comp
-L wickerlib:LED-RGB-WS2812B-4SMD LED5
-U 1 1 595D0515
-P 7890 3650
-F 0 "LED5" H 7940 4025 50  0000 C CNN
-F 1 "WS2812B" H 7940 3934 50  0000 C CNN
-F 2 "002:WS2812B" H 7890 3300 50  0001 C CIN
-F 3 "http://www.adafruit.com/datasheets/WS2812B.pdf" H 7890 3650 5   0001 C CNN
-F 4 "LED RGB WS2812B W/DVR 4SMD" H 7890 3300 50  0001 C CIN "Description"
-F 5 "Adafruit" H 7890 3300 50  0001 C CIN "MF_Name"
-F 6 "1655" H 7890 3300 50  0001 C CIN "MF_PN"
-F 7 "Digikey" H 7890 3300 50  0001 C CIN "S1_Name"
-F 8 "1528-1104-ND" H 7890 3300 50  0001 C CIN "S1_PN"
-	1    7890 3650
-	1    0    0    -1
-$EndComp
-$Comp
-L wickerlib:LED-RGB-WS2812B-4SMD LED4
-U 1 1 595D08CE
-P 6740 3650
-F 0 "LED4" H 6790 4025 50  0000 C CNN
-F 1 "WS2812B" H 6790 3934 50  0000 C CNN
-F 2 "002:WS2812B" H 6740 3300 50  0001 C CIN
-F 3 "http://www.adafruit.com/datasheets/WS2812B.pdf" H 6740 3650 5   0001 C CNN
-F 4 "LED RGB WS2812B W/DVR 4SMD" H 6740 3300 50  0001 C CIN "Description"
-F 5 "Adafruit" H 6740 3300 50  0001 C CIN "MF_Name"
-F 6 "1655" H 6740 3300 50  0001 C CIN "MF_PN"
-F 7 "Digikey" H 6740 3300 50  0001 C CIN "S1_Name"
-F 8 "1528-1104-ND" H 6740 3300 50  0001 C CIN "S1_PN"
-	1    6740 3650
-	1    0    0    -1
-$EndComp
-$Comp
-L wickerlib:LED-RGB-WS2812B-4SMD LED3
-U 1 1 595D1904
-P 5465 3650
-F 0 "LED3" H 5515 4025 50  0000 C CNN
-F 1 "WS2812B" H 5515 3934 50  0000 C CNN
-F 2 "002:WS2812B" H 5465 3300 50  0001 C CIN
-F 3 "http://www.adafruit.com/datasheets/WS2812B.pdf" H 5465 3650 5   0001 C CNN
-F 4 "LED RGB WS2812B W/DVR 4SMD" H 5465 3300 50  0001 C CIN "Description"
-F 5 "Adafruit" H 5465 3300 50  0001 C CIN "MF_Name"
-F 6 "1655" H 5465 3300 50  0001 C CIN "MF_PN"
-F 7 "Digikey" H 5465 3300 50  0001 C CIN "S1_Name"
-F 8 "1528-1104-ND" H 5465 3300 50  0001 C CIN "S1_PN"
-	1    5465 3650
-	1    0    0    -1
-$EndComp
-$Comp
-L wickerlib:LED-RGB-WS2812B-4SMD LED2
-U 1 1 595D190F
-P 4215 3650
-F 0 "LED2" H 4265 4025 50  0000 C CNN
-F 1 "WS2812B" H 4265 3934 50  0000 C CNN
-F 2 "002:WS2812B" H 4215 3300 50  0001 C CIN
-F 3 "http://www.adafruit.com/datasheets/WS2812B.pdf" H 4215 3650 5   0001 C CNN
-F 4 "LED RGB WS2812B W/DVR 4SMD" H 4215 3300 50  0001 C CIN "Description"
-F 5 "Adafruit" H 4215 3300 50  0001 C CIN "MF_Name"
-F 6 "1655" H 4215 3300 50  0001 C CIN "MF_PN"
-F 7 "Digikey" H 4215 3300 50  0001 C CIN "S1_Name"
-F 8 "1528-1104-ND" H 4215 3300 50  0001 C CIN "S1_PN"
-	1    4215 3650
-	1    0    0    -1
-$EndComp
-Text GLabel 8805 4360 2    50   Input ~ 0
-+5V
-$Comp
-L pspice:R R1
-U 1 1 597EC094
-P 4320 7610
-F 0 "R1" H 4388 7656 50  0000 L CNN
-F 1 "1k" H 4388 7565 50  0000 L CNN
-F 2 "001:R_1206_HandSoldering" H 4320 7610 50  0001 C CNN
-F 3 "" H 4320 7610 50  0001 C CNN
-	1    4320 7610
-	0    -1   -1   0
-$EndComp
-$Comp
-L NANO33IoTV2.0-rescue:LED-RESCUE-001-001-rescue-HG_002-rescue-001-rescue D1
-U 1 1 597EC09A
-P 4820 7610
-F 0 "D1" V 4860 7430 50  0000 R CNN
-F 1 "ON" V 4770 7435 50  0000 R CNN
-F 2 "002:LED_1206_HandSoldering" H 4820 7610 50  0001 C CNN
-F 3 "" H 4820 7610 50  0001 C CNN
-	1    4820 7610
-	-1   0    0    1
-$EndComp
-Text Label 3970 7610 2    50   ~ 0
-+5V
+P 8455 4435
+F 0 "#PWR0101" H 8455 4185 50  0001 C CNN
+F 1 "GND" H 8460 4262 50  0000 C CNN
+F 2 "" H 8455 4435 50  0001 C CNN
+F 3 "" H 8455 4435 50  0001 C CNN
+	1    8455 4435
+	1    0    0    -1
+$EndComp
 $Comp
 L power:GND #PWR0102
 U 1 1 597EE12E
-P 5070 7610
-F 0 "#PWR0102" H 5070 7360 50  0001 C CNN
-F 1 "GND" H 5075 7437 50  0000 C CNN
-F 2 "" H 5070 7610 50  0001 C CNN
-F 3 "" H 5070 7610 50  0001 C CNN
-	1    5070 7610
+P 5125 7425
+F 0 "#PWR0102" H 5125 7175 50  0001 C CNN
+F 1 "GND" H 5130 7252 50  0000 C CNN
+F 2 "" H 5125 7425 50  0001 C CNN
+F 3 "" H 5125 7425 50  0001 C CNN
+	1    5125 7425
 	1    0    0    -1
 $EndComp
@@
 Wire Wire Line
 	6790 4360 6790 4150
-Wire Wire Line
-	4570 7610 4670 7610
-Wire Wire Line
-	4070 7610 3970 7610
-Wire Wire Line
-	4970 7610 5070 7610
 Wire Wire Line
 	7440 3175 7440 3500
@@
 L power:GND #PWR0103
 U 1 1 59894DC3
-P 8530 4660
-F 0 "#PWR0103" H 8530 4410 50  0001 C CNN
-F 1 "GND" H 8535 4487 50  0000 C CNN
-F 2 "" H 8530 4660 50  0001 C CNN
-F 3 "" H 8530 4660 50  0001 C CNN
-	1    8530 4660
+P 2210 3605
+F 0 "#PWR0103" H 2210 3355 50  0001 C CNN
+F 1 "GND" H 2080 3530 50  0000 C CNN
+F 2 "" H 2210 3605 50  0001 C CNN
+F 3 "" H 2210 3605 50  0001 C CNN
+	1    2210 3605
 	1    0    0    -1
 $EndComp
 Wire Wire Line
 	2490 3500 2415 3500
-Wire Wire Line
-	8440 3900 8640 3900
-Text GLabel 8640 3900 2    50   Input ~ 0
-4-A2
-Text Notes 4200 7095 0    50   ~ 0
+Text Notes 4325 6845 0    50   ~ 0
 POWER LED
 Wire Wire Line
@@
 Wire Wire Line
 	2415 3500 2415 3175
-Text Notes 6505 7120 0    50   ~ 0
+Text Notes 6405 6845 0    50   ~ 0
 Escornabot Art
 Wire Notes Line
 	495  2950 470  2950
 $Comp
-L NANO33IoTV2.0-rescue:HG_SilKs_2-HG-001-rescue SilKs1
+L 001-rescue:HG_SilKs_2-HG SilKs1
 U 1 1 5BD9DD96
-P 6665 7430
-F 0 "SilKs1" H 6843 7476 50  0000 L CNN
-F 1 "Escorni_Art" H 6843 7385 50  0000 L CNN
-F 2 "002-Nano:escorni-badge-new_05_Nano_100mm" H 6665 7430 50  0001 C CNN
-F 3 "" H 6665 7430 50  0001 C CNN
-	1    6665 7430
-	1    0    0    -1
-$EndComp
-$Comp
-L wickerlib:LED-RGB-WS2812B-4SMD LED1
-U 1 1 595D1F1E
-P 2940 3650
-F 0 "LED1" H 2990 4025 50  0000 C CNN
-F 1 "WS2812B" H 2990 3934 50  0000 C CNN
-F 2 "002:WS2812B" H 2940 3300 50  0001 C CIN
-F 3 "http://www.adafruit.com/datasheets/WS2812B.pdf" H 2940 3650 5   0001 C CNN
-	1    2940 3650
-	1    0    0    -1
-$EndComp
-NoConn ~ 2390 3900
-Connection ~ 7940 4360
+P 6565 7155
+F 0 "SilKs1" H 6743 7201 50  0000 L CNN
+F 1 "Escorni_Art" H 6743 7110 50  0000 L CNN
+F 2 "002-Nano:escorni-badge-new_05_Nano_100mm" H 6565 7155 50  0001 C CNN
+F 3 "" H 6565 7155 50  0001 C CNN
+	1    6565 7155
+	1    0    0    -1
+$EndComp
 $Comp
 L Device:C C1
 U 1 1 5D6867E5
-P 8530 4510
-F 0 "C1" H 8645 4556 50  0000 L CNN
-F 1 "22nF" H 8645 4465 50  0000 L CNN
-F 2 "002:C_1206_HandSoldering" H 8568 4360 50  0001 C CNN
-F 3 "~" H 8530 4510 50  0001 C CNN
-	1    8530 4510
-	1    0    0    -1
-$EndComp
-Connection ~ 8530 4360
-Wire Wire Line
-	8530 4360 8805 4360
-Wire Wire Line
-	7940 4360 8530 4360
+P 2210 3420
+F 0 "C1" H 1900 3485 50  0000 L CNN
+F 1 "22nF" H 1900 3390 50  0000 L CNN
+F 2 "002:C_1206_HandSoldering" H 2248 3270 50  0001 C CNN
+F 3 "~" H 2210 3420 50  0001 C CNN
+	1    2210 3420
+	1    0    0    -1
+$EndComp
 Wire Wire Line
 	2415 3175 2210 3175
@@
 Text Label 8975 1075 2    50   ~ 0
 A2
+$Comp
+L Device:R R1
+U 1 1 5D69DAF4
+P 4425 7375
+F 0 "R1" V 4218 7375 50  0000 C CNN
+F 1 "1k" V 4309 7375 50  0000 C CNN
+F 2 "Resistor_SMD:R_0805_2012Metric_Pad1.15x1.40mm_HandSolder" V 4355 7375 50  0001 C CNN
+F 3 "~" H 4425 7375 50  0001 C CNN
+	1    4425 7375
+	0    1    1    0
+$EndComp
+$Comp
+L Device:LED D1
+U 1 1 5D69E441
+P 4850 7375
+F 0 "D1" H 4843 7120 50  0000 C CNN
+F 1 "LED" H 4843 7211 50  0000 C CNN
+F 2 "LED_SMD:LED_0805_2012Metric_Pad1.15x1.40mm_HandSolder" H 4850 7375 50  0001 C CNN
+F 3 "~" H 4850 7375 50  0001 C CNN
+	1    4850 7375
+	-1   0    0    1
+$EndComp
+Wire Wire Line
+	5000 7375 5125 7375
+Wire Wire Line
+	5125 7375 5125 7425
+Wire Wire Line
+	4575 7375 4700 7375
+Wire Wire Line
+	4275 7375 4150 7375
+Text GLabel 10225 1475 2    50   Input ~ 0
+NEO-D3
+Wire Wire Line
+	9975 1475 10225 1475
+Text GLabel 2390 3900 0    50   Input ~ 0
+NEO-D3
+Text Label 2065 3175 2    50   ~ 0
++3V3
+Wire Wire Line
+	2210 3175 2210 3270
+$Comp
+L NANO33IoTV2.0-rescue:WS2812B LED1
+U 1 1 5D6E7F3D
+P 2940 3650
+F 0 "LED1" H 2990 4025 50  0000 C CNN
+F 1 "WS2812B" H 2990 3934 50  0000 C CNN
+F 2 "002:WS2812B" H 2940 2700 50  0001 C CIN
+F 3 "" H 2940 3650 5   0001 C CNN
+F 4 "LED RGB WS2812B" H 2940 2600 50  0001 C CIN "Description"
+	1    2940 3650
+	1    0    0    -1
+$EndComp
+$Comp
+L NANO33IoTV2.0-rescue:WS2812B LED2
+U 1 1 5D6EAB0C
+P 4215 3650
+F 0 "LED2" H 4265 4025 50  0000 C CNN
+F 1 "WS2812B" H 4265 3934 50  0000 C CNN
+F 2 "002:WS2812B" H 4215 2700 50  0001 C CIN
+F 3 "" H 4215 3650 5   0001 C CNN
+F 4 "LED RGB WS2812B" H 4215 2600 50  0001 C CIN "Description"
+	1    4215 3650
+	1    0    0    -1
+$EndComp
+$Comp
+L NANO33IoTV2.0-rescue:WS2812B LED5
+U 1 1 5D6EB699
+P 7890 3650
+F 0 "LED5" H 7940 4025 50  0000 C CNN
+F 1 "WS2812B" H 7940 3934 50  0000 C CNN
+F 2 "002:WS2812B" H 7890 2700 50  0001 C CIN
+F 3 "" H 7890 3650 5   0001 C CNN
+F 4 "LED RGB WS2812B" H 7890 2600 50  0001 C CIN "Description"
+	1    7890 3650
+	1    0    0    -1
+$EndComp
+$Comp
+L NANO33IoTV2.0-rescue:WS2812B LED4
+U 1 1 5D6EC20A
+P 6740 3650
+F 0 "LED4" H 6790 4025 50  0000 C CNN
+F 1 "WS2812B" H 6790 3934 50  0000 C CNN
+F 2 "002:WS2812B" H 6740 2700 50  0001 C CIN
+F 3 "" H 6740 3650 5   0001 C CNN
+F 4 "LED RGB WS2812B" H 6740 2600 50  0001 C CIN "Description"
+	1    6740 3650
+	1    0    0    -1
+$EndComp
+$Comp
+L NANO33IoTV2.0-rescue:WS2812B LED3
+U 1 1 5D6EC9B7
+P 5465 3650
+F 0 "LED3" H 5515 4025 50  0000 C CNN
+F 1 "WS2812B" H 5515 3934 50  0000 C CNN
+F 2 "002:WS2812B" H 5465 2700 50  0001 C CIN
+F 3 "" H 5465 3650 5   0001 C CNN
+F 4 "LED RGB WS2812B" H 5465 2600 50  0001 C CIN "Description"
+	1    5465 3650
+	1    0    0    -1
+$EndComp
+Wire Wire Line
+	2210 3175 2065 3175
+Connection ~ 2210 3175
+Wire Wire Line
+	2210 3570 2210 3605
+Wire Wire Line
+	7940 4360 8455 4360
+Wire Wire Line
+	8455 4360 8455 4435
+Connection ~ 7940 4360
+NoConn ~ 8440 3900
+Text Notes 8685 1670 0    79   ~ 0
+?
+Text Notes 8710 705  0    79   ~ 0
+?
+Text Notes 8750 1990 0    79   ~ 0
+?
+Text Label 4150 7375 2    50   ~ 0
++3V3
 $EndSCHEMATC

Commit message: Add some minors changes
Parts:
- C1: footprint 002:C_1206_HandSoldering -> Capacitor_SMD:C_0805_2012Metric_Pad1.15x1.40mm_HandSolder
- J1: footprint Arduino:NANO_33_Socket_Castell -> Arduino:NANO_33_Single_Socket
Other:
- note added: "Normaly NC"
- note added: "Power Out"
- note removed: "?"
- moved on the sheet: J1
