File: Regla-Leds/001/001.kicad_pcb (KiCad board)
At the start: 2 copper layers, 49.7 x 49.3 mm, 14 parts, among them J2 Conn_01x08

Commit message: Add route trace
Parts:
- removed Ref**: Val**, Reverse_Mount_Leds:Regla_Leds
- removed svg2mod: G***, Reverse_Mount_Leds:Firma.2019.CuMask.01
- added U1: PCB, Reverse_Mount_Leds:Regla_Leds, F.Cu at (158.8, 92.7)
- turned C2 to 270 degrees
- turned LED2 to 180 degrees
Connections:
- net /VCC renamed VCC
Routing:
- net VCC: track 0.00 -> 81.5 mm
- net /Port_C: track 0.00 -> 49.0 mm
- net /Port_B: track 0.00 -> 26.8 mm, vias 0 -> 2
- net Net-(D2-Pad2): track 0.00 -> 22.8 mm, vias 0 -> 2
- net /Port_A: track 0.00 -> 21.9 mm
- net Net-(D1-Pad2): track 0.00 -> 21.9 mm
- net GND: track 0.00 -> 9.47 mm, vias 0 -> 6
- net /Led_2: track 0.00 -> 9.43 mm, vias 0 -> 2
- net Net-(D3-Pad2): track 0.00 -> 4.48 mm
- net /Led_1: track 0.00 -> 3.81 mm
- net /Led_3: track 0.00 -> 3.79 mm
- added copper zone on B.Cu, net GND
- added copper zone on F.Cu, net GND

Commit message: Moonlight soldering Kit Updates
Parts:
- added G***: LOGO, Reverse_Mount_Leds:OSHpark-2-1800, B.Cu at (145.9, 82.7)
- added PP-G***: PP-LOGO, Reverse_Mount_Leds:OSHpark-1-1200, B.Cu at (146.3, 78.0)
- added REF***: OSHW-Logo2_7.3x6mm_SilkScreen, Reverse_Mount_Leds:OSHW-Logo2_7.3x6mm_SilkScreen, B.Cu at (160.0, 93.5)
- added svg2mod: G***, Reverse_Mount_Leds:firma_Cu_Mask, B.Cu at (174.2, 103.6)
- moved LED3 0.39 mm to (166.9, 75.1)
- moved J2 0.15 mm to (147.5, 113.4)
Routing:
- net VCC: track 81.5 -> 78.3 mm
- net /Port_C: track 49.0 -> 47.7 mm
- net GND: track 9.47 -> 10.2 mm, vias 6 -> 5
Other:
- board text added: ""Moonlight" The reverse mount soldering kit."
- board text added: "Developed By"
- board text removed: "The reverse LED welding practice kit."
