File: Regla-Leds/001/001.sch (KiCad schematic (older format))
At the start: 13 parts, among them J2 Conn_01x08, U1 PCB

Commit message: Add route trace
Changed lines of the file:
@@
 Wire Wire Line
 	10325 1125 10325 1000
-Text Label 10325 1000 2    50   ~ 0
-VCC
 Wire Wire Line
 	5925 3450 5775 3450
@@
 	1    0    0    -1
 $EndComp
+$Comp
+L power:VCC #PWR09
+U 1 1 5D91B027
+P 10325 1000
+F 0 "#PWR09" H 10325 850 50  0001 C CNN
+F 1 "VCC" H 10342 1173 50  0000 C CNN
+F 2 "" H 10325 1000 50  0001 C CNN
+F 3 "" H 10325 1000 50  0001 C CNN
+	1    10325 1000
+	1    0    0    -1
+$EndComp

Commit message: Moonlight soldering Kit Updates
Parts:
- added U2: Firma, Reverse_Mount_Leds:firma_Cu_Mask, symbol Reverse_mount_leds:PCB
Changed lines of the file:
@@
+	1    0    0    -1
+$EndComp
+$Comp
+L Reverse_mount_leds:PCB U2
+U 1 1 5D927C25
+P 7650 3675
+F 0 "U2" H 7749 3721 50  0000 L CNN
+F 1 "Firma" H 7749 3630 50  0000 L CNN
+F 2 "Reverse_Mount_Leds:firma_Cu_Mask" H 7650 3675 50  0001 C CNN
+F 3 "" H 7650 3675 50  0001 C CNN
+	1    7650 3675
 	1    0    0    -1
 $EndComp

Commit message: Check
Parts:
- LED1, LED2, LED3: symbol Reverse_mount_leds:WS2812B-Normal -> 001-rescue:WS2812B-Normal-Reverse_mount_leds
- U1, U2: symbol Reverse_mount_leds:PCB -> 001-rescue:PCB-Reverse_mount_leds
Changed lines of the file:
@@
 $EndDescr
 $Comp
-L Reverse_mount_leds:WS2812B-Normal LED1
+L 001-rescue:WS2812B-Normal-Reverse_mount_leds LED1
 U 1 1 5D90F91C
 P 4450 1575
@@
 VCC
 $Comp
-L Reverse_mount_leds:WS2812B-Normal LED2
+L 001-rescue:WS2812B-Normal-Reverse_mount_leds LED2
 U 1 1 5D91778C
 P 6050 1575
@@
 	6100 2075 6100 2200
 $Comp
-L Reverse_mount_leds:WS2812B-Normal LED3
+L 001-rescue:WS2812B-Normal-Reverse_mount_leds LED3
 U 1 1 5D91A7C4
 P 7600 1575
@@
 $EndComp
 $Comp
-L Reverse_mount_leds:PCB U1
+L 001-rescue:PCB-Reverse_mount_leds U1
 U 1 1 5D912D99
 P 7650 3450
@@
 $EndComp
 $Comp
-L Reverse_mount_leds:PCB U2
+L 001-rescue:PCB-Reverse_mount_leds U2
 U 1 1 5D927C25
 P 7650 3675
