File: Regla-Leds/Varios_Leds/001.kicad_pcb (KiCad board)
At the start: 2 copper layers, 49.7 x 49.3 mm, 17 parts, among them J2 Conn_01x08, U1 PCB

Commit message: Minor changes MoonLigth
Routing:
- net VCC: track 79.5 -> 78.3 mm
