File: Attiny_Wearable/001/Tiny.sch (KiCad schematic (older format))
At the start: 18 parts, among them SW1 SW_Push, SW2 SW_Push_SPDT, U1 ATtiny85-20SU

Commit message: some minors updates
Parts:
- BT1: symbol Device:Battery_3V_Coin -> Tiny-rescue:Battery_3V_Coin-Device
Changed lines of the file:
@@
 $EndComp
 $Comp
-L Device:Battery_3V_Coin BT1
+L Tiny-rescue:Battery_3V_Coin-Device BT1
 U 1 1 5D584BA9
 P 4300 3500
