File: Regla-Leds/Charly_Plex/001.sch (KiCad schematic (older format))
At the start: 9 parts, among them J1 Conn_01x09, U1 PCB, U2 Firma

Commit message: Add Digispark Footprint
Parts:
- removed J1: Conn_01x09, Reverse_Mount_Leds:Digispark_SMD, symbol Connector_Generic:Conn_01x09
- added J2: Conn_01x06_x03, Reverse_Mount_Leds:Digispark_SMD_Reverse, symbol Digispark:Conn_01x06_x03
Connections:
- net GND: now also J2.8 (GND)
- net VCC: now also J2.9 (5V)
- net VIN: now also J2.7 (VIn)
- net Led_1 renamed PB_0
- net PB_0: now also J2.1 (P0_D0)
- net Led_2 renamed PB_1
- net PB_1: now also J2.2 (P1_D1)
- net Led_3 renamed PB_4
- net PB_4: now also J2.5 (P4_D4)
- no-connect marks 0 -> 3
Other:
- note added: "Charlie Plexing"
- note removed: "Leds"
- moved on the sheet: U1, U2
Changed lines of the file:
@@
 L power:PWR_FLAG #FLG01
 U 1 1 5D92F7A7
-P 9750 1025
-F 0 "#FLG01" H 9750 1100 50  0001 C CNN
-F 1 "PWR_FLAG" H 9750 1198 50  0000 C CNN
-F 2 "" H 9750 1025 50  0001 C CNN
-F 3 "~" H 9750 1025 50  0001 C CNN
-	1    9750 1025
+P 6325 1500
+F 0 "#FLG01" H 6325 1575 50  0001 C CNN
+F 1 "PWR_FLAG" H 6325 1673 50  0000 C CNN
+F 2 "" H 6325 1500 50  0001 C CNN
+F 3 "~" H 6325 1500 50  0001 C CNN
+	1    6325 1500
 	1    0    0    -1
 $EndComp
@@
 L power:GND #PWR04
 U 1 1 5D930D3A
-P 9750 1150
-F 0 "#PWR04" H 9750 900 50  0001 C CNN
-F 1 "GND" H 9755 977 50  0000 C CNN
-F 2 "" H 9750 1150 50  0001 C CNN
-F 3 "" H 9750 1150 50  0001 C CNN
-	1    9750 1150
-	1    0    0    -1
-$EndComp
-Wire Wire Line
-	9750 1025 9750 1150
+P 6325 1625
+F 0 "#PWR04" H 6325 1375 50  0001 C CNN
+F 1 "GND" H 6330 1452 50  0000 C CNN
+F 2 "" H 6325 1625 50  0001 C CNN
+F 3 "" H 6325 1625 50  0001 C CNN
+	1    6325 1625
+	1    0    0    -1
+$EndComp
+Wire Wire Line
+	6325 1500 6325 1625
 $Comp
 L power:PWR_FLAG #FLG02
 U 1 1 5D932C92
-P 10325 1125
-F 0 "#FLG02" H 10325 1200 50  0001 C CNN
-F 1 "PWR_FLAG" H 10325 1298 50  0000 C CNN
-F 2 "" H 10325 1125 50  0001 C CNN
-F 3 "~" H 10325 1125 50  0001 C CNN
-	1    10325 1125
+P 6900 1600
+F 0 "#FLG02" H 6900 1675 50  0001 C CNN
+F 1 "PWR_FLAG" H 6900 1773 50  0000 C CNN
+F 2 "" H 6900 1600 50  0001 C CNN
+F 3 "~" H 6900 1600 50  0001 C CNN
+	1    6900 1600
 	-1   0    0    1
 $EndComp
 Wire Wire Line
-	10325 1125 10325 1000
-Wire Wire Line
-	5925 3450 5775 3450
-Wire Wire Line
-	5925 3550 5775 3550
-Wire Wire Line
-	5925 3650 5775 3650
-Wire Wire Line
-	5925 3750 5775 3750
-Text Label 5775 4050 2    50   ~ 0
+	6900 1600 6900 1475
+Text Label 4725 1800 2    50   ~ 0
 VIN
 $Comp
 L power:GND #PWR05
 U 1 1 5D93CBC2
-P 5525 4300
-F 0 "#PWR05" H 5525 4050 50  0001 C CNN
-F 1 "GND" H 5530 4127 50  0000 C CNN
-F 2 "" H 5525 4300 50  0001 C CNN
-F 3 "" H 5525 4300 50  0001 C CNN
-	1    5525 4300
-	1    0    0    -1
-$EndComp
-Text Label 5775 3450 2    50   ~ 0
-Port_A
-Text Label 5775 3550 2    50   ~ 0
-Port_B
-Text Label 5775 3650 2    50   ~ 0
-Port_C
-Text Notes 1725 850  0    79   ~ 0
-Leds
+P 4450 1775
+F 0 "#PWR05" H 4450 1525 50  0001 C CNN
+F 1 "GND" H 4455 1602 50  0000 C CNN
+F 2 "" H 4450 1775 50  0001 C CNN
+F 3 "" H 4450 1775 50  0001 C CNN
+	1    4450 1775
+	1    0    0    -1
+$EndComp
+Text Label 5150 2375 3    50   ~ 0
+PB_0
+Text Label 5250 2375 3    50   ~ 0
+PB_1
+Text Label 5350 2375 3    50   ~ 0
+PB_2
+Text Notes 1925 900  0    79   ~ 0
+Charlie Plexing
 $Comp
 L Device:LED D1
@@
 	0    1    1    0
 $EndComp
-Text Label 1175 1125 2    50   ~ 0
-Led_1
-Text Label 1175 1700 2    50   ~ 0
-Led_2
-Text Label 1175 2275 2    50   ~ 0
-Led_3
 $Comp
 L 001-rescue:PCB-Reverse_mount_leds U1
 U 1 1 5D912D99
-P 7650 3450
-F 0 "U1" H 7749 3496 50  0000 L CNN
-F 1 "PCB" H 7749 3405 50  0000 L CNN
-F 2 "Reverse_Mount_Leds:Regla_Leds" H 7650 3450 50  0001 C CNN
-F 3 "" H 7650 3450 50  0001 C CNN
-	1    7650 3450
+P 7900 1425
+F 0 "U1" H 7999 1471 50  0000 L CNN
+F 1 "PCB" H 7999 1380 50  0000 L CNN
+F 2 "Reverse_Mount_Leds:Regla_Leds" H 7900 1425 50  0001 C CNN
+F 3 "" H 7900 1425 50  0001 C CNN
+	1    7900 1425
 	1    0    0    -1
 $EndComp
@@
 L power:VCC #PWR09
 U 1 1 5D91B027
-P 10325 1000
-F 0 "#PWR09" H 10325 850 50  0001 C CNN
-F 1 "VCC" H 10342 1173 50  0000 C CNN
-F 2 "" H 10325 1000 50  0001 C CNN
-F 3 "" H 10325 1000 50  0001 C CNN
-	1    10325 1000
+P 6900 1475
+F 0 "#PWR09" H 6900 1325 50  0001 C CNN
+F 1 "VCC" H 6917 1648 50  0000 C CNN
+F 2 "" H 6900 1475 50  0001 C CNN
+F 3 "" H 6900 1475 50  0001 C CNN
+	1    6900 1475
 	1    0    0    -1
 $EndComp
@@
 L 001-rescue:PCB-Reverse_mount_leds U2
 U 1 1 5D927C25
-P 7650 3675
-F 0 "U2" H 7749 3721 50  0000 L CNN
-F 1 "Firma" H 7749 3630 50  0000 L CNN
-F 2 "Reverse_Mount_Leds:firma_Cu_Mask" H 7650 3675 50  0001 C CNN
-F 3 "" H 7650 3675 50  0001 C CNN
-	1    7650 3675
-	1    0    0    -1
-$EndComp
-$Comp
-L Connector_Generic:Conn_01x09 J1
-U 1 1 5D99DEAA
-P 6125 3850
-F 0 "J1" H 6205 3892 50  0000 L CNN
-F 1 "Conn_01x09" H 6205 3801 50  0000 L CNN
-F 2 "Reverse_Mount_Leds:Digispark_SMD" H 6125 3850 50  0001 C CNN
-F 3 "~" H 6125 3850 50  0001 C CNN
-	1    6125 3850
-	1    0    0    -1
-$EndComp
-Wire Wire Line
-	5925 3850 5775 3850
-Wire Wire Line
-	5925 3950 5775 3950
-Wire Wire Line
-	5925 4050 5775 4050
-Text Label 5775 4250 2    50   ~ 0
+P 7900 1650
+F 0 "U2" H 7999 1696 50  0000 L CNN
+F 1 "Firma" H 7999 1605 50  0000 L CNN
+F 2 "Reverse_Mount_Leds:firma_Cu_Mask" H 7900 1650 50  0001 C CNN
+F 3 "" H 7900 1650 50  0001 C CNN
+	1    7900 1650
+	1    0    0    -1
+$EndComp
+Text Label 4725 1600 2    50   ~ 0
 VCC
 $Comp
@@
 Wire Wire Line
 	3725 1125 3725 1525
-Text Label 5775 3750 2    50   ~ 0
-Port_D
-Text Label 5775 3850 2    50   ~ 0
-Port_E
-Text Label 5775 3950 2    50   ~ 0
-Port_F
-Wire Wire Line
-	5525 4150 5525 4300
-Wire Wire Line
-	5525 4150 5925 4150
-Wire Wire Line
-	5925 4250 5775 4250
+Text Label 5450 2375 3    50   ~ 0
+PB_3
+Text Label 5550 2375 3    50   ~ 0
+PB_4
+Text Label 5650 2375 3    50   ~ 0
+PB_5
 $Comp
 L power:PWR_FLAG #FLG03
 U 1 1 5DA04141
-P 10900 1125
-F 0 "#FLG03" H 10900 1200 50  0001 C CNN
-F 1 "PWR_FLAG" H 10900 1298 50  0000 C CNN
-F 2 "" H 10900 1125 50  0001 C CNN
-F 3 "~" H 10900 1125 50  0001 C CNN
-	1    10900 1125
+P 7475 1600
+F 0 "#FLG03" H 7475 1675 50  0001 C CNN
+F 1 "PWR_FLAG" H 7475 1773 50  0000 C CNN
+F 2 "" H 7475 1600 50  0001 C CNN
+F 3 "~" H 7475 1600 50  0001 C CNN
+	1    7475 1600
 	-1   0    0    1
 $EndComp
 Wire Wire Line
-	10900 1125 10900 1000
+	7475 1600 7475 1475
 $Comp
 L wickerlib:VIN #PWR01
 U 1 1 5DA054F6
-P 10900 1000
-F 0 "#PWR01" H 10900 850 50  0001 C CNN
-F 1 "VIN" H 10915 1173 50  0000 C CNN
-F 2 "" H 10900 1000 50  0000 C CNN
-F 3 "" H 10900 1000 50  0000 C CNN
-	1    10900 1000
-	1    0    0    -1
-$EndComp
+P 7475 1475
+F 0 "#PWR01" H 7475 1325 50  0001 C CNN
+F 1 "VIN" H 7490 1648 50  0000 C CNN
+F 2 "" H 7475 1475 50  0000 C CNN
+F 3 "" H 7475 1475 50  0000 C CNN
+	1    7475 1475
+	1    0    0    -1
+$EndComp
+$Comp
+L Digispark:Conn_01x06_x03 J2
+U 1 1 5DA5B104
+P 5350 2050
+F 0 "J2" H 5300 3175 50  0000 L CNN
+F 1 "Conn_01x06_x03" V 5800 2050 50  0001 L CNN
+F 2 "Reverse_Mount_Leds:Digispark_SMD_Reverse" H 4825 1000 50  0001 C CNN
+F 3 "~" H 4825 1000 50  0001 C CNN
+	1    5350 2050
+	1    0    0    -1
+$EndComp
+Wire Wire Line
+	4850 1600 4725 1600
+Wire Wire Line
+	4850 1800 4725 1800
+Wire Wire Line
+	5150 2250 5150 2375
+Wire Wire Line
+	5250 2250 5250 2375
+Wire Wire Line
+	5550 2250 5550 2375
+Wire Wire Line
+	4450 1700 4450 1775
+Wire Wire Line
+	4450 1700 4850 1700
+Text Label 1175 1125 2    50   ~ 0
+PB_0
+Text Label 1175 1700 2    50   ~ 0
+PB_1
+Text Label 1175 2275 2    50   ~ 0
+PB_4
+NoConn ~ 5350 2250
+NoConn ~ 5450 2250
+NoConn ~ 5650 2250
 $EndSCHEMATC
