File: Nano_33/template/001/001.kicad_pcb (KiCad board)
At the start: 2 copper layers, 17.8 x 43.2 mm, 8 parts, among them P1 Digital, P2 Analog, P3 CONN_01X01, P4 CONN_01X01, P5 CONN_01X01, P6 CONN_01X01

Commit message: Add Cylon Badge
Parts:
- added REF**: TFT_0.96_SPI, Display:TFT_0.96_SPI, F.Cu at (145.6, 91.6)
Changed lines of the file:
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@@
-(kicad_pcb (version 20171130) (host pcbnew 5.1.2-f72e74a~84~ubuntu18.04.1)
+(kicad_pcb (version 20171130) (host pcbnew 5.1.4-e60b266~84~ubuntu18.04.1)
   (general
     (thickness 1.6)
@@
     (tracks 0)
     (zones 0)
-    (modules 8)
+    (modules 9)
     (nets 33)
   )
@@
     (add_net "Net-(P6-Pad1)")
   )
+  (module Display:TFT_0.96_SPI (layer F.Cu)
+    (at 145.5674 91.6178)
+    (fp_text reference REF** (at 0 3.937) (layer F.Fab)
+      (effects (font (size 1 1) (thickness 0.15)))
+    )
+    (fp_text value TFT_0.96_SPI (at 0 -5.969) (layer F.Fab)
+      (effects (font (size 1 1) (thickness 0.15)))
+    )
+    (fp_text user 13 (at 5.1435 2.0955) (layer F.Fab)
+      (effects (font (size 0.8 0.8) (thickness 0.15)))
+    )
+    (fp_text user 1 (at -4.7625 2.0955) (layer F.Fab)
+      (effects (font (size 0.8 0.8) (thickness 0.15)))
+    )
+    (fp_line (start -6.7945 -15.0495) (end -6.7945 13.6505) (layer F.Fab) (width 0.12))
+    (fp_line (start -6.7945 -15.0495) (end 6.7755 -15.0495) (layer F.Fab) (width 0.12))
+    (fp_line (start 6.7755 13.6525) (end -6.7945 13.6525) (layer F.Fab) (width 0.12))
+    (fp_line (start 6.7755 13.6525) (end 6.7755 -15.0475) (layer F.Fab) (width 0.12))
+    (fp_line (start 5.334 -1.651) (end -5.334 -1.651) (layer F.Fab) (width 0.12))
+    (fp_line (start -6.35 -0.635) (end -6.35 4.064) (layer F.Fab) (width 0.12))
+    (fp_line (start -4.5085 6.096) (end -4.5085 12.2555) (layer F.Fab) (width 0.12))
+    (fp_line (start -3.4925 13.2715) (end 3.429 13.2715) (layer F.Fab) (width 0.12))
+    (fp_line (start 4.445 12.2555) (end 4.445 6.1595) (layer F.Fab) (width 0.12))
+    (fp_line (start 6.35 4.1275) (end 6.35 -0.635) (layer F.Fab) (width 0.12))
+    (fp_arc (start -5.334 4.064) (end -6.35 4.064) (angle -90) (layer F.Fab) (width 0.12))
+    (fp_arc (start -5.334 -0.635) (end -5.334 -1.651) (angle -90) (layer F.Fab) (width 0.12))
+    (fp_arc (start 5.334 -0.635) (end 6.35 -0.635) (angle -90) (layer F.Fab) (width 0.12))
+    (fp_arc (start 5.334 4.1275) (end 5.334 5.1435) (angle -90) (layer F.Fab) (width 0.12))
+    (fp_arc (start 5.461 6.1595) (end 5.461 5.1435) (angle -90) (layer F.Fab) (width 0.12))
+    (fp_arc (start 3.429 12.2555) (end 3.429 13.2715) (angle -90) (layer F.Fab) (width 0.12))
+    (fp_arc (start -3.4925 12.2555) (end -4.5085 12.2555) (angle -90) (layer F.Fab) (width 0.12))
+    (fp_arc (start -5.5245 6.096) (end -4.5085 6.096) (angle -90) (layer F.Fab) (width 0.12))
+    (pad 1 smd rect (at -4.2 0) (size 0.4 2.4) (layers F.Cu F.Paste F.Mask))
+    (pad 13 smd rect (at 4.2 0) (size 0.4 2.4) (layers F.Cu F.Paste F.Mask))
+    (pad 2 smd rect (at -3.5 0) (size 0.4 2.4) (layers F.Cu F.Paste F.Mask))
+    (pad 7 smd rect (at 0 0) (size 0.4 2.4) (layers F.Cu F.Paste F.Mask))
+    (pad 3 smd rect (at -2.8 0) (size 0.4 2.4) (layers F.Cu F.Paste F.Mask))
+    (pad 4 smd rect (at -2.1 0) (size 0.4 2.4) (layers F.Cu F.Paste F.Mask))
+    (pad 5 smd rect (at -1.4 0) (size 0.4 2.4) (layers F.Cu F.Paste F.Mask))
+    (pad 6 smd rect (at -0.7 0) (size 0.4 2.4) (layers F.Cu F.Paste F.Mask))
+    (pad 11 smd rect (at 2.8 0) (size 0.4 2.4) (layers F.Cu F.Paste F.Mask))
+    (pad 8 smd rect (at 0.7 0) (size 0.4 2.4) (layers F.Cu F.Paste F.Mask))
+    (pad 9 smd rect (at 1.4 0) (size 0.4 2.4) (layers F.Cu F.Paste F.Mask))
+    (pad 12 smd rect (at 3.5 0) (size 0.4 2.4) (layers F.Cu F.Paste F.Mask))
+    (pad 10 smd rect (at 2.1 0) (size 0.4 2.4) (layers F.Cu F.Paste F.Mask))
+  )
   (module template:Socket_Strip_Arduino_1x15 (layer F.Cu)
