File: Reverse-Leds/Charly_Plex_6_Leds_Ala_Gaviota_Moon_75mm/001.kicad_pcb (KiCad board)
At the start: 2 copper layers, 73.9 x 73.2 mm, 14 parts, among them J1 Conn_01x02, J2 Conn_01x06_x03, U1 PCB, U2 Firma

Commit message: UpdateMoon
Parts:
- removed G***: LOGO, Reverse_Mount_Leds:OSHpark-2-1800
- removed PP-G***: PP-LOGO, Reverse_Mount_Leds:OSHpark-1-1200
- removed REF***: OSHW-Logo2_7.3x6mm_SilkScreen, Reverse_Mount_Leds:OSHW-Logo2_7.3x6mm_SilkScreen
- added U3: Oshpark_logo, Reverse_Mount_Leds:OSHpark-1-1200, B.Cu at (129.3, 90.3)
- added U4: Oshpark_Purple, Reverse_Mount_Leds:OSHpark-2-1800, B.Cu at (128.9, 95.4)
- added U5: OSHW_Silk, Symbol:OSHW-Logo2_9.8x8mm_SilkScreen, B.Cu at (166.1, 107.8)
- turned J1 to 180 degrees
Connections:
- BT1 pad 1: VIN -> VCC
- J1 pad 1: VIN -> VCC
Routing:
- net VIN: track 106.2 -> 0.00 mm, vias 4 -> 0
- net VCC: track 0.00 -> 95.5 mm, vias 0 -> 4
- net GND: vias 5 -> 7

Commit message: Add Attiny85 Breakout
Parts:
- added R1: R_Small, Resistor_SMD:R_1206_3216Metric_Pad1.42x1.75mm_HandSolder, B.Cu at (145.4, 127.6)
- added SW2: SW_Push_Dual, Moon_75mm_Gaviota:SW_Push_PTS647_4.5mm, B.Cu at (154.9, 132.1)
- BT1: footprint Battery:S8211R -> Moon_75mm_Gaviota:S8211R
- D1, D2, D3, D4, D5, D6: footprint Reverse_Mount_Leds:SunLed_PLCC_Reverse-2 -> Moon_75mm_Gaviota:SunLed_PLCC_Reverse-2
- J1: footprint Connector_JST:JST-S2B-PH-SM4-TB -> Moon_75mm_Gaviota:JST-S2B-PH-SM4-TB
- J2: footprint Reverse_Mount_Leds:Digispark_SMD_Reverse -> Moon_75mm_Gaviota:Digispark_SMD_Reverse
- U1: footprint Reverse_Mount_Leds:Moon_6_Leds_75_2 -> Moon_75mm_Gaviota:Moon_6_Leds_75_2
- U2: footprint Reverse_Mount_Leds:firma_Cu_Mask -> Moon_75mm_Gaviota:firma_Cu_Mask
- U3: footprint Reverse_Mount_Leds:OSHpark-1-1200 -> Moon_75mm_Gaviota:OSHpark-1-1200
- U4: footprint Reverse_Mount_Leds:OSHpark-2-1800 -> Moon_75mm_Gaviota:OSHpark-2-1800
- moved U5 37.2 mm to (129.3, 112.7)
- moved U2 16.2 mm to (138.0, 134.0)
Connections:
- J2 pad 3: Net-(J2-Pad3) -> /PB_2
Routing:
- net /PB_2: track 0.00 -> 38.7 mm
- net VCC: track 95.5 -> 111.2 mm
- net /PB_1: track 84.9 -> 82.2 mm
- net /PB_4: track 88.1 -> 90.3 mm
- net /PB_0: track 90.7 -> 90.8 mm, vias 0 -> 2
- net GND: vias 7 -> 8
Other:
- board text added: "Fly me to the moon Let me play among the stars And let me see what spring is like On a-Jupiter and Mars In other words, hold my hand In other words, baby, kiss me"

Commit message: Add Cylon Badge
Parts:
- added Ref**: Val**, Moon_75mm_Gaviota:Moon_ATtiny85, F.Cu at (196.2, 104.8)
