File: Cylon/Cylon_New_Charly_Plex_6_75mm/001.sch (KiCad schematic (older format))
At the start: 17 parts, among them J1 Conn_01x02, J2 Conn_01x06_x03, SW2 SW_Push_Dual, U1 PCB, U2 Firma, U3 Oshpark_logo, U4 Oshpark_Purple, U5 OSHW_Silk, U6 Love_ATtiny85

Commit message: New_Install_SO_Update
Changed lines of the file:
@@
 EESchema Schematic File Version 4
-LIBS:001-cache
 EELAYER 30 0
 EELAYER END
@@
 	10750 1250 10750 1125
 $Comp
-L wickerlib:VIN #PWR01
+L 001-rescue:VIN-wickerlib #PWR01
 U 1 1 5DA054F6
 P 10750 1125
