File: Cylon/Cylon_New_Charly_Plex_6_75mm/001.kicad_pcb (KiCad board)
At the start: 2 copper layers, 58.8 x 74.3 mm, 17 parts, among them J1 Conn_01x02, J2 Conn_01x06_x03, SW2 SW_Push_Dual, U1 PCB, U2 Firma, U3 Oshpark_logo, U4 Oshpark_Purple, U5 OSHW_Silk, U6 Love_ATtiny85

Commit message: Add agora Pin 2032
Parts:
- added BT1: Battery_Cell, Cylon_New_Charly_Plex_6_75mm:S8211R, F.Cu at (228.6, 74.3)
Changed lines of the file:
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@@
   (general
     (thickness 1.6)
-    (drawings 0)
+    (drawings 2)
     (tracks 1)
     (zones 0)
-    (modules 17)
+    (modules 18)
     (nets 10)
   )
@@
     (uvia_drill 0.508)
   )
+  (module Cylon_New_Charly_Plex_6_75mm:S8211R (layer F.Cu)
+    (at 228.6 74.295)
+    (fp_text reference BT1 (at 10.16 12.446) (layer F.Fab)
+      (effects (font (size 1 1) (thickness 0.15)))
+    )
+    (fp_text value Battery_Cell (at -9.398 -10.16) (layer F.Fab)
+      (effects (font (size 1 1) (thickness 0.15)))
+    )
+    (fp_line (start 12.8 -9.1) (end 12.8 10.9) (layer F.Fab) (width 0.15))
+    (fp_line (start -12.8 -9.1) (end 12.8 -9.1) (layer F.Fab) (width 0.15))
+    (fp_line (start -12.8 10.9) (end -12.8 -9.1) (layer F.Fab) (width 0.15))
+    (fp_line (start 12.8 10.9) (end -12.8 10.9) (layer F.Fab) (width 0.15))
+    (pad 1 smd rect (at 12.8 0) (size 5.5 5.5) (layers F.Cu F.Paste F.Mask)
+      (net 2 VCC))
+    (pad 1 smd rect (at -12.8 0) (size 5.5 5.5) (layers F.Cu F.Paste F.Mask)
+      (net 2 VCC))
+    (pad 2 smd rect (at 0 0) (size 4 4) (layers F.Cu F.Paste F.Mask)
+      (net 1 GND))
+    (model ${KISYS3DMOD}/Battery.3dshapes/s8211-46r.stp
+      (offset (xyz 0 6 4))
+      (scale (xyz 1 1 1))
+      (rotate (xyz 90 90 180))
+    )
+    (model ${KISYS3DMOD}/Battery.3dshapes/CR-2032-01.step
+      (offset (xyz 0 0 3.5))
+      (scale (xyz 1 1 1))
+      (rotate (xyz 90 0 0))
+    )
+  )
   (module Cylon_New_Charly_Plex_6_75mm:S8211R (layer B.Cu)
     (at 154.686 81.788)
@@
       (xy -20.920506 17.504971) (xy -20.912666 17.504834) (xy -20.834337 17.516996)) (layer B.Mask) (width 0.01))
   )
+  (dimension 23.495 (width 0.1524) (layer F.SilkS)
+    (gr_text "23.495 mm" (at 249.6058 73.3425 90) (layer F.SilkS)
+      (effects (font (size 1.016 1.016) (thickness 0.1524)))
+    )
+    (feature1 (pts (xy 215.9 61.595) (xy 248.871421 61.595)))
+    (feature2 (pts (xy 215.9 85.09) (xy 248.871421 85.09)))
+    (crossbar (pts (xy 248.285 85.09) (xy 248.285 61.595)))
+    (arrow1a (pts (xy 248.285 61.595) (xy 248.871421 62.721504)))
+    (arrow1b (pts (xy 248.285 61.595) (xy 247.698579 62.721504)))
+    (arrow2a (pts (xy 248.285 85.09) (xy 248.871421 83.963496)))
+    (arrow2b (pts (xy 248.285 85.09) (xy 247.698579 83.963496)))
+  )
+  (dimension 31.75 (width 0.1524) (layer F.SilkS)
+    (gr_text "31.750 mm" (at 228.6 95.9358) (layer F.SilkS)
+      (effects (font (size 1.016 1.016) (thickness 0.1524)))
+    )
+    (feature1 (pts (xy 212.725 77.47) (xy 212.725 95.201421)))
+    (feature2 (pts (xy 244.475 77.47) (xy 244.475 95.201421)))
+    (crossbar (pts (xy 244.475 94.615) (xy 212.725 94.615)))
+    (arrow1a (pts (xy 212.725 94.615) (xy 213.851504 94.028579)))
+    (arrow1b (pts (xy 212.725 94.615) (xy 213.851504 95.201421)))
+    (arrow2a (pts (xy 244.475 94.615) (xy 243.348496 94.028579)))
+    (arrow2b (pts (xy 244.475 94.615) (xy 243.348496 95.201421)))
+  )
   (via (at 154.71394 81.71688) (size 0.6858) (drill 0.3302) (layers F.Cu B.Cu) (net 1))
   (zone (net 1) (net_name GND) (layer F.Cu) (hatch edge 0.508)
     (connect_pads (clearance 0.508))
     (min_thickness 0.254)
-    (fill yes (arc_segments 32) (thermal_gap 0.508) (thermal_bridge_width 0.508))
+    (fill (arc_segments 32) (thermal_gap 0.508) (thermal_bridge_width 0.508))
     (polygon
       (pts
@@
     (connect_pads (clearance 0.508))
     (min_thickness 0.254)
-    (fill yes (arc_segments 32) (thermal_gap 0.508) (thermal_bridge_width 0.508))
+    (fill (arc_segments 32) (thermal_gap 0.508) (thermal_bridge_width 0.508))
     (polygon
       (pts

Commit message: New_Install_SO_Update
Parts:
- removed the BT1 at (228.6, 74.3)
- moved U6 19.6 mm to (175.8, 112.8)
Routing:
- net VCC: track 0.00 -> 131.0 mm
- net /PB_0: track 0.00 -> 41.7 mm
- net /PB_2: track 0.00 -> 40.6 mm
- net /PB_1: track 0.00 -> 39.1 mm, vias 0 -> 4
- net /PB_4: track 0.00 -> 34.4 mm

Commit message: Some changes
Parts:
- moved D1 1.48 mm to (163.3, 97.5), turned to 320 degrees
- moved D3 1.42 mm to (152.4, 102.9), turned to 80 degrees
- moved D4 1.25 mm to (156.5, 102.8), turned to 280 degrees
- moved D6 0.90 mm to (144.9, 97.0), turned to 40 degrees
- moved D2 0.90 mm to (160.7, 99.7), turned to 130 degrees
- moved D5 0.90 mm to (148.0, 99.7), turned to 230 degrees
Routing:
- net /PB_4: track 34.4 -> 61.2 mm, vias 0 -> 2
- net /PB_1: track 39.1 -> 50.6 mm, vias 4 -> 0
- net /PB_0: track 41.7 -> 51.4 mm
- net GND: vias 1 -> 0
