File: Feather_To_NANO_Breakout/Feather/FeatherWing_KC5.kicad_pcb (KiCad board)
At the start: 2 copper layers, 43.2 x 22.9 mm, 4 parts, among them J1 feather long, J2 feather short, J3 Conn_01x15, J4 Conn_01x15

Commit message: Update
Minor changes
Parts:
- added G***Ki: Ki-LOGO, Feather_Nano_Brealout:Ki-2500, B.Cu at (152.9, 91.3)
- added G***Ki: Ki-LOGO, Feather_Nano_Brealout:Ki-2500, F.Cu at (152.9, 91.2)
- added REF***: OSHW-Logo2_7.3x6mm_SilkScreen, Feather_Nano_Brealout:OSHW-Logo2_7.3x6mm_SilkScreen, B.Cu at (145.6, 91.4)
- added REF***: OSHW-Logo2_7.3x6mm_SilkScreen, Feather_Nano_Brealout:OSHW-Logo2_7.3x6mm_SilkScreen, F.Cu at (145.5, 91.3)
- added Ref**: Val**, Feather_Nano_Brealout:Moon_The_Shield_SilkS, B.Cu at (124.6, 91.6)
- added Ref**: Val**, Feather_Nano_Brealout:Moon_Firma_SilkS, B.Cu at (133.7, 91.0)
- added Ref**: Val**, Feather_Nano_Brealout:Moon_The_Shield_SilkS, F.Cu at (127.0, 91.7)
- added Ref**: Val**, Feather_Nano_Brealout:Moon_Firma_SilkS, F.Cu at (134.5, 91.0)
- added Ref**: Val**, Feather_Nano_Brealout:Feather_Silks, F.Cu at (141.5, 91.4)
- added Ref**: Val**, Feather_Nano_Brealout:Feather_CU, B.Cu at (161.8, 91.9)
- added Ref**: Val**, Feather_Nano_Brealout:Feather_CU, F.Cu at (161.8, 92.6)
Routing:
- net GND: track 12.8 -> 10.5 mm
- net /SCK-D13: track 32.4 -> 31.2 mm
- net /TX: track 19.3 -> 18.3 mm
- net /SCL-A5: track 28.4 -> 27.6 mm
Other:
- board text removed: "3V3"
- board text removed: "A0"
- board text removed: "A1"
- board text removed: "A2"
- board text removed: "A3"
- board text removed: "A4"
- board text removed: "A5"
- board text removed: "AREF"
- board text removed: "FREE"
- board text removed: "GND"
- board text removed: "MISO"
- board text removed: "MOSI"
- board text removed: "NC"
- board text removed: "RX"
- board text removed: "SCK"
- board text removed: "TX"
- board text removed: "VUSB"
- board text removed: "~RST"
