File: tft-shield/MKR-100-1010-TFT/MKRWiFi1010V2.0.sch (KiCad schematic (older format))
At the start: 1 part

Commit message: Some minors updates
Parts:
- J?: symbol MKR-Familiy:MKR-1000 -> MKRWiFi1010V2.0-rescue:MKR-1000-MKR-Familiy
Changed lines of the file:
@@
 EESchema Schematic File Version 4
-LIBS:MKRWiFi1010V2.0-cache
 EELAYER 30 0
 EELAYER END
@@
 $EndDescr
 $Comp
-L MKR-Familiy:MKR-1000 J?
+L MKRWiFi1010V2.0-rescue:MKR-1000-MKR-Familiy J?
 U 1 1 5DAEEFF7
 P 10275 1475
