File: tft-shield/TFT_MKR_1000/001.kicad_pcb (KiCad board)
At the start: 2 copper layers, 35.6 x 22.9 mm, 8 parts, among them J1 MKR-1000_1010, Q1 S8050, U1 TFT_0.9680*160

Commit message: Some minors updates
Other:
- board size 35.6 x 22.9 mm -> 36.8 x 22.9 mm
Changed lines of the file:
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@@
-(kicad_pcb (version 20171130) (host pcbnew 5.1.4-e60b266~84~ubuntu18.04.1)
+(kicad_pcb (version 20171130) (host pcbnew 5.1.5-52549c5~84~ubuntu18.04.1)
   (general
     (thickness 1.6)
@@
     (47 F.CrtYd user)
     (48 B.Fab user)
-    (49 F.Fab user)
+    (49 F.Fab user hide)
   )
   (setup
-    (last_trace_width 0.3302)
+    (last_trace_width 0.254)
     (user_trace_width 0.1524)
     (user_trace_width 0.254)
@@
     (arrow2b (pts (xy 161.29 113.03) (xy 160.163496 113.616421)))
   )
-  (gr_arc (start 159.385 106.045) (end 159.385 107.95) (angle -90) (layer Edge.Cuts) (width 0.1524))
-  (gr_arc (start 127.635 106.045) (end 125.73 106.045) (angle -90) (layer Edge.Cuts) (width 0.1524))
-  (gr_arc (start 127.635 86.995) (end 127.635 85.09) (angle -90) (layer Edge.Cuts) (width 0.1524))
-  (gr_arc (start 159.385 86.995) (end 161.29 86.995) (angle -90) (layer Edge.Cuts) (width 0.1524))
-  (gr_line (start 161.29 86.995) (end 161.29 106.045) (layer Edge.Cuts) (width 0.1524))
-  (gr_line (start 127.635 85.09) (end 159.385 85.09) (layer Edge.Cuts) (width 0.1524))
-  (gr_line (start 125.73 106.045) (end 125.73 86.995) (layer Edge.Cuts) (width 0.1524))
-  (gr_line (start 159.385 107.95) (end 127.635 107.95) (layer Edge.Cuts) (width 0.1524))
+  (gr_arc (start 160.02 106.045) (end 160.02 107.95) (angle -90) (layer Edge.Cuts) (width 0.1524))
+  (gr_arc (start 127 106.045) (end 125.095 106.045) (angle -90) (layer Edge.Cuts) (width 0.1524))
+  (gr_arc (start 127 86.995) (end 127 85.09) (angle -90) (layer Edge.Cuts) (width 0.1524))
+  (gr_arc (start 160.02 86.995) (end 161.925 86.995) (angle -90) (layer Edge.Cuts) (width 0.1524))
+  (gr_line (start 161.925 86.995) (end 161.925 106.045) (layer Edge.Cuts) (width 0.1524))
+  (gr_line (start 127 85.09) (end 160.02 85.09) (layer Edge.Cuts) (width 0.1524))
+  (gr_line (start 125.095 106.045) (end 125.095 86.995) (layer Edge.Cuts) (width 0.1524))
+  (gr_line (start 160.02 107.95) (end 127 107.95) (layer Edge.Cuts) (width 0.1524))
   (gr_circle (center 117.348 76.962) (end 118.618 76.962) (layer Dwgs.User) (width 0.15))
   (gr_line (start 114.427 78.994) (end 114.427 74.93) (angle 90) (layer Dwgs.User) (width 0.15))
@@
     (connect_pads (clearance 0.508))
     (min_thickness 0.254)
-    (fill (arc_segments 32) (thermal_gap 0.508) (thermal_bridge_width 0.508))
+    (fill yes (arc_segments 32) (thermal_gap 0.508) (thermal_bridge_width 0.508))
     (polygon
       (pts
@@
     (connect_pads (clearance 0.508))
     (min_thickness 0.254)
-    (fill (arc_segments 32) (thermal_gap 0.508) (thermal_bridge_width 0.508))
+    (fill yes (arc_segments 32) (thermal_gap 0.508) (thermal_bridge_width 0.508))
     (polygon
       (pts
