File: Samd11/Breakout_02/001.kicad_pcb (KiCad board)
At the start: 2 copper layers, 20.3 x 19.7 mm, 11 parts, among them IC2 ATSAMD11C14A-SSUT, J1 Conn_01x07, J2 Conn_01x07, U2 Firma

Commit message: Add Star Shield Nano
Parts:
- added J1: USB_A, Connector_USB:USB_A_Plug_PCB, F.Cu at (157.5, 83.2)
Other:
- board size 20.3 x 19.7 mm -> 20.3 x 31.8 mm
Changed lines of the file:
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@@
   (general
     (thickness 1.6)
-    (drawings 13)
+    (drawings 18)
     (tracks 0)
     (zones 0)
-    (modules 11)
+    (modules 12)
     (nets 17)
   )
   (page A4)
   (layers
-    (0 F.Cu signal)
-    (31 B.Cu signal)
-    (32 B.Adhes user)
-    (33 F.Adhes user)
-    (34 B.Paste user)
-    (35 F.Paste user)
-    (36 B.SilkS user)
-    (37 F.SilkS user)
-    (38 B.Mask user)
-    (39 F.Mask user)
-    (40 Dwgs.User user)
-    (41 Cmts.User user)
-    (42 Eco1.User user)
-    (43 Eco2.User user)
+    (0 F.Cu signal hide)
+    (31 B.Cu signal hide)
+    (32 B.Adhes user hide)
+    (33 F.Adhes user hide)
+    (34 B.Paste user hide)
+    (35 F.Paste user hide)
+    (36 B.SilkS user hide)
+    (37 F.SilkS user hide)
+    (38 B.Mask user hide)
+    (39 F.Mask user hide)
+    (40 Dwgs.User user hide)
+    (41 Cmts.User user hide)
+    (42 Eco1.User user hide)
+    (43 Eco2.User user hide)
     (44 Edge.Cuts user)
-    (45 Margin user)
+    (45 Margin user hide)
     (46 B.CrtYd user)
     (47 F.CrtYd user)
@@
     (add_net "Net-(D2-Pad1)")
   )
+  (module Connector_USB:USB_A_Plug_PCB (layer F.Cu)
+    (at 157.48 83.185 180)
+    (attr virtual)
+    (fp_text reference J1 (at 0.13 -7.85 180) (layer F.SilkS) hide
+      (effects (font (size 1.5 1.5) (thickness 0.15)))
+    )
+    (fp_text value USB_A (at 0.29 -10.13 180) (layer F.SilkS) hide
+      (effects (font (size 1.5 1.5) (thickness 0.15)))
+    )
+    (fp_line (start 6.03 0) (end 6.03 -12) (layer Dwgs.User) (width 0.15))
+    (fp_line (start 6.03 0) (end -6.03 0) (layer Dwgs.User) (width 0.15))
+    (fp_line (start -6.03 0) (end -6.03 -12) (layer Dwgs.User) (width 0.15))
+    (pad 1 connect rect (at 3.81 -4.9 180) (size 1.9 8) (layers F.Cu F.Mask))
+    (pad 4 connect rect (at -3.81 -4.9 180) (size 1.9 8) (layers F.Cu F.Mask))
+    (pad 3 connect rect (at -1.3 -5.15 180) (size 2 7.5) (layers F.Cu F.Mask))
+    (pad 2 connect rect (at 1.3 -5.15 180) (size 2 7.5) (layers F.Cu F.Mask))
+  )
   (module SamD11_Breakout:Back_SAMD11 (layer F.Cu)
     (at 157.6578 105.7402)
@@
     )
   )
+  (gr_line (start 163.5125 83.185) (end 163.5125 95.245) (layer Edge.Cuts) (width 0.15))
+  (gr_line (start 151.4525 83.19) (end 151.4525 95.25) (layer Edge.Cuts) (width 0.15))
+  (dimension 12.06 (width 0.15) (layer Dwgs.User)
+    (gr_text "12.060 mm" (at 157.48 80.8182) (layer Dwgs.User)
+      (effects (font (size 1 1) (thickness 0.15)))
+    )
+    (feature1 (pts (xy 163.51 83.185) (xy 163.51 81.531779)))
+    (feature2 (pts (xy 151.45 83.185) (xy 151.45 81.531779)))
+    (crossbar (pts (xy 151.45 82.1182) (xy 163.51 82.1182)))
+    (arrow1a (pts (xy 163.51 82.1182) (xy 162.383496 82.704621)))
+    (arrow1b (pts (xy 163.51 82.1182) (xy 162.383496 81.531779)))
+    (arrow2a (pts (xy 151.45 82.1182) (xy 152.576504 82.704621)))
+    (arrow2b (pts (xy 151.45 82.1182) (xy 152.576504 81.531779)))
+  )
+  (gr_line (start 151.4525 83.185) (end 163.5125 83.185) (layer Edge.Cuts) (width 0.15))
+  (gr_line (start 163.5125 95.25) (end 165.735 95.25) (layer Edge.Cuts) (width 0.15))
   (gr_text "Developed\nby" (at 162.0774 105.156 90) (layer B.SilkS)
     (effects (font (size 0.8 0.8) (thickness 0.2)) (justify mirror))
@@
     (arrow2b (pts (xy 148.59 88.265) (xy 149.716504 87.678579)))
   )
-  (gr_arc (start 149.225 97.155) (end 149.225 95.25) (angle -90) (layer Edge.Cuts) (width 0.05))
+  (gr_arc (start 149.225 97.155) (end 149.225 95.25) (angle -90) (layer Edge.Cuts) (width 0.15))
   (dimension 8.89 (width 0.12) (layer F.Fab)
     (gr_text "8.890 mm" (at 153.035 118.11) (layer F.Fab)
@@
     (arrow2b (pts (xy 148.59 116.84) (xy 149.716504 116.253579)))
   )
-  (gr_line (start 147.32 113.03) (end 147.32 97.155) (layer Edge.Cuts) (width 0.05))
-  (gr_arc (start 149.225 113.03) (end 147.32 113.03) (angle -90) (layer Edge.Cuts) (width 0.05))
-  (gr_line (start 165.735 114.935) (end 149.225 114.935) (layer Edge.Cuts) (width 0.05))
-  (gr_arc (start 165.735 113.03) (end 165.735 114.935) (angle -90) (layer Edge.Cuts) (width 0.05))
-  (gr_arc (start 165.735 97.155) (end 167.64 97.155) (angle -90) (layer Edge.Cuts) (width 0.05))
-  (gr_line (start 167.64 97.155) (end 167.64 113.03) (layer Edge.Cuts) (width 0.05))
-  (gr_line (start 149.225 95.25) (end 165.735 95.25) (layer Edge.Cuts) (width 0.05))
+  (gr_line (start 147.32 113.03) (end 147.32 97.155) (layer Edge.Cuts) (width 0.15))
+  (gr_arc (start 149.225 113.03) (end 147.32 113.03) (angle -90) (layer Edge.Cuts) (width 0.15))
+  (gr_line (start 165.735 114.935) (end 149.225 114.935) (layer Edge.Cuts) (width 0.15))
+  (gr_arc (start 165.735 113.03) (end 165.735 114.935) (angle -90) (layer Edge.Cuts) (width 0.15))
+  (gr_arc (start 165.735 97.155) (end 167.64 97.155) (angle -90) (layer Edge.Cuts) (width 0.15))
+  (gr_line (start 167.64 97.155) (end 167.64 113.03) (layer Edge.Cuts) (width 0.15))
+  (gr_line (start 149.225 95.25) (end 151.4525 95.25) (layer Edge.Cuts) (width 0.15))
 )
