File: Lober/001/001.kicad_pcb (KiCad board)
At the start: 2 copper layers, 0 parts

Commit message: Update lober
Parts:
- added BT1: Battery_3V_Coin, lober:WA-BCMC, B.Cu at (145.4, 101.6)
- added REF**: LED_SK6812_EC15_1.5x1.5mm, LED_SMD:LED_SK6812_EC15_1.5x1.5mm, F.Cu at (160.7, 92.1)
- added REF**: LED_SK6812_EC15_1.5x1.5mm, LED_SMD:LED_SK6812_EC15_1.5x1.5mm, F.Cu at (145.4, 118.7)
- added REF**: LED_SK6812_EC15_1.5x1.5mm, LED_SMD:LED_SK6812_EC15_1.5x1.5mm, F.Cu at (129.5, 92.1)
- added Ref**: Val**, lober:lober, F.Cu at (145.4, 104.8)
Other:
- board outline added: 49.3 x 45 mm
