File: Feather_To_NANO_Breakout/1.- NANO to Feather Rev 1 w-lipo/FeatherWing_KC5.sch (KiCad schematic (older format))
At the start: 17 parts, among them J1 feather long, J2 feather short, J3 Conn_01x15, J4 Conn_01x15, J5 Conn_01x02, U1 Feather_Cu, U10 Feather_Silks, U11 KiCadLogo, U2 Feather_Silks, U3 KiCadLogo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

Commit message: Update gitignore
Parts:
- U1, U10, U11, U2, U3, U4, U5, U6, U7, U8, U9: symbol Graphic:Extra -> FeatherWing_KC5-rescue:Extra-Graphic
Changed lines of the file:
@@
 NoConn ~ 4675 4850
 $Comp
-L Graphic:Extra U1
+L FeatherWing_KC5-rescue:Extra-Graphic U1
 U 1 1 5E2BEF7F
 P 7075 1800
@@
 $EndComp
 $Comp
-L Graphic:Extra U2
+L FeatherWing_KC5-rescue:Extra-Graphic U2
 U 1 1 5E2BF776
 P 7075 2100
@@
 $EndComp
 $Comp
-L Graphic:Extra U3
+L FeatherWing_KC5-rescue:Extra-Graphic U3
 U 1 1 5E2BFB4E
 P 7075 2400
@@
 $EndComp
 $Comp
-L Graphic:Extra U4
+L FeatherWing_KC5-rescue:Extra-Graphic U4
 U 1 1 5E2C0E92
 P 7075 2700
@@
 $EndComp
 $Comp
-L Graphic:Extra U5
+L FeatherWing_KC5-rescue:Extra-Graphic U5
 U 1 1 5E2C0E9C
 P 7075 3000
@@
 $EndComp
 $Comp
-L Graphic:Extra U6
+L FeatherWing_KC5-rescue:Extra-Graphic U6
 U 1 1 5E2C0EA6
 P 7075 3300
@@
 VIN
 $Comp
-L Graphic:Extra U7
+L FeatherWing_KC5-rescue:Extra-Graphic U7
 U 1 1 5E2696B4
 P 7925 1775
@@
 $EndComp
 $Comp
-L Graphic:Extra U8
+L FeatherWing_KC5-rescue:Extra-Graphic U8
 U 1 1 5E269B67
 P 7950 2400
@@
 $EndComp
 $Comp
-L Graphic:Extra U9
+L FeatherWing_KC5-rescue:Extra-Graphic U9
 U 1 1 5E26B47E
 P 7950 2700
@@
 $EndComp
 $Comp
-L Graphic:Extra U10
+L FeatherWing_KC5-rescue:Extra-Graphic U10
 U 1 1 5E26CA20
 P 7950 3000
@@
 $EndComp
 $Comp
-L Graphic:Extra U11
+L FeatherWing_KC5-rescue:Extra-Graphic U11
 U 1 1 5E26D0ED
 P 7950 3300
